File: uHoubolt_PCB_FCU/uHoubolt_PCB_FCU.sch (KiCad schematic (older format))
At the start: 122 parts, among them J1 206832-0202, J2 206832-0202, J3 206832-0202, Q1 BSB008NE2LX, Q2 BSB008NE2LX, Q3 BSB008NE2LX, U1 INA180, U2 INA180, U3 INA180

Commit message: Implemented changes after design review
Parts:
- removed C? (x3): 0.1u, symbol Device:C_Small
- removed C?: 10n, symbol Device:C_Small
- removed F? (x3): Polyfuse, symbol Device:Polyfuse
- removed J? (x3): JST GH, symbol Connector_Generic_MountingPin:Conn_01x04_MountingPin
- removed J? (x2): 206832-0202, symbol Connector_Generic:Conn_01x02
- removed JP?: SolderJumper_3_Open, symbol Jumper:SolderJumper_3_Open
- removed Q? (x2): BSB008NE2LX, Package_DirectFET:DirectFET_MX, symbol Transistor_FET:BSB008NE2LX
- removed R?: 3.3k/0, symbol Device:R_Small
- removed R?: 6.8k/160, symbol Device:R_Small
- removed R? (x2): 5m 1W, symbol Device:R_Small
- removed R? (x6): 47k, symbol Device:R_Small
- removed R? (x6): 33k, symbol Device:R_Small
- removed R? (x4): 20k, symbol Device:R_Small
- removed R? (x2): 200, symbol Device:R_Small
- removed R? (x2): 200k, symbol Device:R_Small
- removed R? (x2): 56k, symbol Device:R_Small
- removed R? (x2): 10k, symbol Device:R_Small
- removed U? (x6): INA180, Package_TO_SOT_SMD:SOT-23-6, symbol TXV_LIB:INA180
- removed U? (x3): AD8426, symbol SCB-rescue:AD8426-TXV_Library_Symbols
- added C2, C24, C25, C26: 100n, symbol Device:C_Small
- added D1: RB218NS-60TL, symbol Device:D_Schottky_x2_KCom_KAA
- added F1, F2, F3: C1H15 (15A fuse), symbol Device:Fuse_Small
- added J11: Conn_01x02, symbol Connector_Generic:Conn_01x02
- added J17, J18: 206832-0202, symbol Connector_Generic:Conn_01x02
- added J2, J7, J9: JST GH, symbol Connector_Generic_MountingPin:Conn_01x04_MountingPin
- added J8: Conn_01x04, symbol Connector_Generic:Conn_01x04
- added JP2: SolderJumper_3_Open, symbol Jumper:SolderJumper_3_Open
- added NT1: Net-Tie_2, symbol Device:Net-Tie_2
- added Q4, Q5: BSB008NE2LX, Package_DirectFET:DirectFET_MX, symbol Transistor_FET:BSB008NE2LX
- added R10, R18, R7: 33k, symbol Device:R_Small
- added R11, R16, R37, R38, R8: 20k, symbol Device:R_Small
- added R17, R6, R9: 47k, symbol Device:R_Small
- added R27, R46, R47: 10k, symbol Device:R_Small
- added R29, R32: 4.7k, symbol Device:R_Small
- added R30, R31: 6.8k, symbol Device:R_Small
- added R4: 4.7k/0, symbol Device:R_Small
- added R40, R41: 200, symbol Device:R_Small
- added R43, R44: 5m 1W, symbol Device:R_Small
- added R5: 6.8k/160, symbol Device:R_Small
- added R50, R52: 200k, symbol Device:R_Small
- added R51, R53: 56k, symbol Device:R_Small
- added U10, U11, U8, U9: INAx180x2 (50V/V gain), Package_TO_SOT_SMD:SOT-23-6, symbol TXV_LIB:INA180
- added U4, U5: INAx180x1 (20V/V gain), Package_TO_SOT_SMD:SOT-23-6, symbol TXV_LIB:INA180
- C1, C21, C27, C3, C4, C5: renamed from C?; value 0.1u -> 100n
- C19: renamed from C1; value 0.1u -> 100n
- C20: renamed from C2; value 0.1u -> 100n
- C23: renamed from C3; value 0.1u -> 100n
- L1: renamed from L?; value 1.5m -> 5.3u
- R13: renamed from R?; value 3.3k -> 4.7k
- R2: renamed from R?; value 3.3k/0 -> 4.7k/0
- U1: renamed from U?; value INA180 -> INAx180x1 (20V/V gain)
- U2, U3: value INA180 -> INAx180x1 (20V/V gain)
- U7: renamed from U1; value INA180 -> INAx180x2 (50V/V gain)
- gave numbers to parts that had none: 39
- renumbered J1 to J14, J2 to J15, J3 to J16, R2 to R24, R3 to R25, R1 to R28, R5 to R33, R6 to R34, R8 to R36, R9 to R39, R11 to R48, R10 to R49
Connections:
- net +3V3: now also C21.1, C2.1, C24.1, C25.1, C26.2, R46.2, R47.2, U10.6 (V+), U11.6 (V+), U4.6 (V+), U5.6 (V+), U8.6 (V+), U9.6 (V+); no longer C21.2
- net +5V: now also JP2.1 (A)
- net +7.5V: now also J7.3 (Pin_3), J9.3 (Pin_3), R31.1
- net GND: now also C12.2, C13.2, C14.1, C15.2, C17.2, C21.2, C6.1, C7.2, U6.13 (P_GND), U6.27 (P_GND_PAD), U6.3 (P_GND), U6.4 (P_GND), C2.2, C24.2, C25.2, C26.1, J11.1 (Pin_1), J2.4 (Pin_4), J2.MP (MountPin), J7.4 (Pin_4), J7.MP (MountPin), J8.1 (Pin_1), J9.4 (Pin_4), J9.MP (MountPin), NT1.2, R10.1, R11.2, R16.1, R18.1, R30.2, R32.2, R37.1, R38.1, R43.2, R44.2, R5.2, R51.2, R53.2, R7.1, R8.1, U10.2 (GND), U10.4 (-), U11.2 (GND), U11.4 (-), U4.2 (GND), U5.2 (GND), U8.2 (GND), U8.4 (-), U9.2 (GND), U9.4 (-); no longer C21.1, U2.4 (-), U3.4 (-)
- net IGNITECONTINUITY2: now also R50.2, R51.1
- net IGNITECONTINUITY3: now also R52.2, R53.1
- net IGNITECONTROL2: now also R37.2, R40.1
- net IGNITECONTROL3: now also R38.2, R41.1
- net IGNITESENSE1: now also U9.1; no longer U3.1
- net IGNITESENSE2: now also U10.1
- net IGNITESENSE3: now also U11.1
- net PRESSURESENSE1: now also U3.1
- net PRESSURESENSE2: now also U4.1
- net PRESSURESENSE3: now also U5.1
- net SERVO2_PWM: now also J7.2 (Pin_2), R8.2
- net SERVO3_PWM: now also J9.2 (Pin_2), R16.2
- net SOLSENSE2: now also U8.1; no longer U2.1
- net TESTPRESSURESENSE2: now also U2.1, R4.2, R5.1
- net VOLTREG_EN: now also R11.1
- net Vdrive: now also F1.1, F2.1, F3.1, J11.2 (Pin_2), R46.1, R47.1; no longer C6.2, C7.1, C8.1, U6.1 (V_IN), U6.2 (V_IN), U6.22 (V_IN), U6.26 (V_IN_PAD)
- net at J14.2 (Pin_2), Q1.1 (D): now also D1.3 (A)
- net at Q2.3 (S), R35.1: now also U8.3 (+); no longer U2.3 (+)
- net at J15.2 (Pin_2), Q2.1 (D): now also D1.2 (A)
- net at Q3.3 (S), R42.1: now also U9.3 (+); no longer U3.3 (+)
- net at J16.1 (Pin_1): now also F1.2
- net at J3.2 (Pin_2): now also U3.3 (+)
- net at J3.3 (Pin_3): now also U3.4 (-)
- net at J4.2 (Pin_2): now also U4.3 (+)
- net at J4.3 (Pin_3): now also U4.4 (-)
- net at J5.2 (Pin_2): now also U5.3 (+)
- net at J5.3 (Pin_3): now also U5.4 (-)
- net at J6.1 (Pin_1): now also R6.2
- net GNDA: now reaches C18.1, R21.2, R23.1, U6.16 (A_GND)
- net GNDA: now also C8.2, U6.25 (A_GND_PAD), NT1.1
- net IMU_INTERRUPT: now reaches U12.6 (INT)
- net at U6.12 (VDRV): now also C14.2; no longer C14.1
- net at U6.14 (P_GOOD): now also R27.1, R29.1
- net at C18.2, R20.1, U6.15 (VDD): now also R27.2
- net +BATT renamed +12V
- net +12V: now also C6.2, C7.1, C8.1, U6.1 (V_IN), U6.2 (V_IN), U6.22 (V_IN), U6.26 (V_IN_PAD), D1.1 (K), J8.4 (Pin_4), JP2.3 (B)
- net SUPPLYMEASURE renamed 5V_SENSE
- new net: J7.1 (Pin_1), R9.2
- new net: J9.1 (Pin_1), R17.2
- new net: J2.1 (Pin_1), JP2.2 (C)
- new net: J2.2 (Pin_2), R4.1, U2.3 (+)
- new net: J2.3 (Pin_3), U2.4 (-)
- new net: J17.2 (Pin_2), Q4.1 (D), R50.1
- new net: Q4.2 (G), R40.2
- new net: Q4.3 (S), R43.1, U10.3 (+)
- new net: F2.2, J17.1 (Pin_1)
- new net: J18.2 (Pin_2), Q5.1 (D), R52.1
- new net: Q5.2 (G), R41.2
- new net: Q5.3 (S), R44.1, U11.3 (+)
- new net: F3.2, J18.1 (Pin_1)
- new net 7V5_SENSE: R31.2, R32.1
- new net SERVO1_FDBK: R6.1, R7.2
- new net SERVO2_FDBK: R10.2, R9.1
- new net SERVO3_FDBK: R17.1, R18.2
- new net VOLTREG_P_GOOD: R29.2, R30.1
- no-connect marks 16 -> 6
Other:
- note added: "(NTC): RC low-pass can use other component values \nif 33u SMD is hard to find"
- note added: "- if using INA180 -> place on high-side of circuit, above MOSFET.\n in case of other OP-AMP: choose one with rail-to-rail amplification!\n- if necessary, replace MOS with another model"
- note added: "7.4V SENSING"
- note added: "BATT3V6"
- note added: "BATT7V2"
- note added: "BATT_GND"
- note added: "BATT_VCC"
- note added: "GND/A_GND NET TIE"
- note added: "PMU Voltage Inputs"
- note added: "connects to PMU connector\nin IGNITION circuit"
- note added: "connects to uHoubold_PCB_PMU\n"J_BALANCE1" connector"
- note added: "keine Elektrolyt-C!\nMan kriegt in Keramik keine 100u"
- note added: "op-amp for diff. 150mV bridge input,\nvoltage div. for 0-5V or 4-20mA input.\n(4.7k/6.8k for 0-5V,\n0/160 Ohm for 4-20mA)"
- note removed: "Vdrive - pyro voltage from PMU\n"
- note removed: "op-amp for diff. 150mV bridge input,\nvoltage div. for 0-5V or 4-20mA input.\n(3.3k/6.8k for 0-5V,\n0/160 Ohm for 4-20mA)"
- moved on the sheet: C10, C12, C13, C14, C15, C17, C18, C21, C22, C6, C7, C8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
