File: PressureSensorInput.sch (KiCad schematic (older format))
At the start: 8 parts, among them J7 Pressure 1, U9 INA180B1

Commit message: preliminary placement done
Parts:
- J7: footprint Connector_JST:JST_GH_SM04B-GHS-TB_1x04-1MP_P1.25mm_Horizontal -> Connector_JST:JST_GH_BM04B-GHS-TBT_1x04-1MP_P1.25mm_Vertical
Changed lines of the file:
@@
 $Descr A4 11693 8268
 encoding utf-8
-Sheet 9 17
+Sheet 2 17
 Title ""
 Date ""
@@
 AR Path="/63D5F044/632B46F4" Ref="#PWR?"  Part="1"
 AR Path="/63DA5A81/632B46F4" Ref="#PWR?"  Part="1"
-F 0 "#PWR0154" H 4975 3925 50  0001 C CNN
+F 0 "#PWR0104" H 4975 3925 50  0001 C CNN
 F 1 "GND" H 4975 4025 50  0000 C CNN
 F 2 "" H 4975 4175 50  0001 C CNN
@@
 AR Path="/63D5F044/632B46FD" Ref="U?"  Part="1"
 AR Path="/63DA5A81/632B46FD" Ref="U?"  Part="1"
-F 0 "U14" H 5775 3675 50  0000 L CNN
+F 0 "U9" H 5775 3675 50  0000 L CNN
 F 1 "INA180B1" H 5625 3600 50  0000 L CNN
 F 2 "Package_TO_SOT_SMD:SOT-23-5" H 5725 3825 50  0001 C CNN
@@
 AR Path="/63D5F044/632B470B" Ref="C?"  Part="1"
 AR Path="/63DA5A81/632B470B" Ref="C?"  Part="1"
-F 0 "C50" V 5825 3450 50  0000 C CNN
+F 0 "C24" V 5825 3450 50  0000 C CNN
 F 1 "100n" V 5600 3450 50  0000 C CNN
 F 2 "Capacitor_SMD:C_0402_1005Metric" H 5725 3450 50  0001 C CNN
@@
 AR Path="/63D5F044/632B4714" Ref="#PWR?"  Part="1"
 AR Path="/63DA5A81/632B4714" Ref="#PWR?"  Part="1"
-F 0 "#PWR0155" H 5575 3850 50  0001 C CNN
+F 0 "#PWR0105" H 5575 3850 50  0001 C CNN
 F 1 "GND" H 5575 3950 50  0000 C CNN
 F 2 "" H 5575 4100 50  0001 C CNN
@@
 AR Path="/63D5F044/632B471B" Ref="R?"  Part="1"
 AR Path="/63DA5A81/632B471B" Ref="R?"  Part="1"
-F 0 "R43" H 5300 4025 50  0000 L CNN
+F 0 "R21" H 5300 4025 50  0000 L CNN
 F 1 "4k7/0" H 5300 3950 50  0000 L CNN
 F 2 "Resistor_SMD:R_0603_1608Metric" H 5250 4000 50  0001 C CNN
@@
 AR Path="/63D5F044/632B4721" Ref="R?"  Part="1"
 AR Path="/63DA5A81/632B4721" Ref="R?"  Part="1"
-F 0 "R44" H 5300 4250 50  0000 L CNN
+F 0 "R22" H 5300 4250 50  0000 L CNN
 F 1 "6k8/160" H 5300 4175 50  0000 L CNN
 F 2 "Resistor_SMD:R_0603_1608Metric" H 5250 4250 50  0001 C CNN
@@
 AR Path="/63D5F044/632B4727" Ref="#PWR?"  Part="1"
 AR Path="/63DA5A81/632B4727" Ref="#PWR?"  Part="1"
-F 0 "#PWR0156" H 5250 4125 50  0001 C CNN
+F 0 "#PWR0106" H 5250 4125 50  0001 C CNN
 F 1 "GND" H 5250 4225 50  0000 C CNN
 F 2 "" H 5250 4375 50  0001 C CNN
@@
 AR Path="/63D5F044/632B472F" Ref="JP?"  Part="1"
 AR Path="/63DA5A81/632B472F" Ref="JP?"  Part="1"
-F 0 "JP6" H 5200 3630 50  0000 C CNN
+F 0 "JP1" H 5200 3630 50  0000 C CNN
 F 1 "V_SEL" H 5200 3539 50  0000 C CNN
 F 2 "Jumper:SolderJumper-3_P1.3mm_Open_RoundedPad1.0x1.5mm" H 5200 3425 50  0001 C CNN
@@
 AR Path="/63D5F044/632B4738" Ref="J?"  Part="1"
 AR Path="/63DA5A81/632B4738" Ref="J?"  Part="1"
-F 0 "J14" H 5050 3725 50  0000 L CNN
+F 0 "J7" H 5050 3725 50  0000 L CNN
 F 1 "Pressure 1" H 5050 3625 50  0000 L CNN
-F 2 "Connector_JST:JST_GH_SM04B-GHS-TB_1x04-1MP_P1.25mm_Horizontal" H 4975 3725 50  0001 C CNN
+F 2 "Connector_JST:JST_GH_BM04B-GHS-TBT_1x04-1MP_P1.25mm_Vertical" H 4975 3725 50  0001 C CNN
 F 3 "~" H 4975 3725 50  0001 C CNN
 	1    4975 3725
@@
 AR Path="/63D5F044/632B4744" Ref="#PWR?"  Part="1"
 AR Path="/63DA5A81/632B4744" Ref="#PWR?"  Part="1"
-F 0 "#PWR0157" H 5850 3200 50  0001 C CNN
+F 0 "#PWR0107" H 5850 3200 50  0001 C CNN
 F 1 "GND" V 5850 3250 50  0000 C CNN
 F 2 "" H 5850 3450 50  0001 C CNN
@@
 AR Path="/63D5F044/632B4751" Ref="R?"  Part="1"
 AR Path="/63DA5A81/632B4751" Ref="R?"  Part="1"
-F 0 "R45" V 6050 3825 50  0000 R CNN
+F 0 "R23" V 6050 3825 50  0000 R CNN
 F 1 "9k1" V 6200 3850 50  0000 R CNN
 F 2 "Resistor_SMD:R_0603_1608Metric" H 6125 3775 50  0001 C CNN
@@
 AR Path="/63D5F044/632B475B" Ref="#PWR?"  Part="1"
 AR Path="/63DA5A81/632B475B" Ref="#PWR?"  Part="1"
-F 0 "#PWR0158" H 6275 3775 50  0001 C CNN
+F 0 "#PWR0108" H 6275 3775 50  0001 C CNN
 F 1 "GND" H 6275 3875 50  0000 C CNN
 F 2 "" H 6275 4025 50  0001 C CNN
@@
 AR Path="/63D5F044/632B4765" Ref="C?"  Part="1"
 AR Path="/63DA5A81/632B4765" Ref="C?"  Part="1"
-F 0 "C51" H 6050 3925 50  0000 L CNN
+F 0 "C41" H 6050 3925 50  0000 L CNN
 F 1 "100n" H 6075 3825 50  0000 L CNN
 F 2 "Capacitor_SMD:C_0402_1005Metric" H 6275 3900 50  0001 C CNN
@@
 AR Path="/63D5F044/632B476B" Ref="#PWR?"  Part="1"
 AR Path="/63DA5A81/632B476B" Ref="#PWR?"  Part="1"
-F 0 "#PWR0159" H 5400 3200 50  0001 C CNN
+F 0 "#PWR0109" H 5400 3200 50  0001 C CNN
 F 1 "+12V" H 5400 3500 50  0000 C CNN
 F 2 "" H 5400 3350 50  0001 C CNN
@@
 AR Path="/63D5F044/632B4771" Ref="#PWR?"  Part="1"
 AR Path="/63DA5A81/632B4771" Ref="#PWR?"  Part="1"
-F 0 "#PWR0160" H 5575 3275 50  0001 C CNN
+F 0 "#PWR0110" H 5575 3275 50  0001 C CNN
 F 1 "+3V3" H 5575 3575 50  0000 C CNN
 F 2 "" H 5575 3425 50  0001 C CNN
@@
 AR Path="/63D5F044/632B4777" Ref="#PWR?"  Part="1"
 AR Path="/63DA5A81/632B4777" Ref="#PWR?"  Part="1"
-F 0 "#PWR0161" H 5000 3200 50  0001 C CNN
+F 0 "#PWR0111" H 5000 3200 50  0001 C CNN
 F 1 "+5V" H 5000 3500 50  0000 C CNN
 F 2 "" H 5000 3350 50  0001 C CNN

Commit message: moved 7V4 buck to separate board
Changed lines of the file:
@@
 AR Path="/63D5F044/632B46FD" Ref="U?"  Part="1"
 AR Path="/63DA5A81/632B46FD" Ref="U?"  Part="1"
-F 0 "U9" H 5775 3675 50  0000 L CNN
+F 0 "U15" H 5775 3675 50  0000 L CNN
 F 1 "INA180B1" H 5625 3600 50  0000 L CNN
 F 2 "Package_TO_SOT_SMD:SOT-23-5" H 5725 3825 50  0001 C CNN
@@
 AR Path="/63D5F044/632B470B" Ref="C?"  Part="1"
 AR Path="/63DA5A81/632B470B" Ref="C?"  Part="1"
-F 0 "C24" V 5825 3450 50  0000 C CNN
+F 0 "C52" V 5825 3450 50  0000 C CNN
 F 1 "100n" V 5600 3450 50  0000 C CNN
 F 2 "Capacitor_SMD:C_0402_1005Metric" H 5725 3450 50  0001 C CNN
@@
 AR Path="/63D5F044/632B471B" Ref="R?"  Part="1"
 AR Path="/63DA5A81/632B471B" Ref="R?"  Part="1"
-F 0 "R21" H 5300 4025 50  0000 L CNN
+F 0 "R46" H 5300 4025 50  0000 L CNN
 F 1 "4k7/0" H 5300 3950 50  0000 L CNN
 F 2 "Resistor_SMD:R_0603_1608Metric" H 5250 4000 50  0001 C CNN
@@
 AR Path="/63D5F044/632B4721" Ref="R?"  Part="1"
 AR Path="/63DA5A81/632B4721" Ref="R?"  Part="1"
-F 0 "R22" H 5300 4250 50  0000 L CNN
+F 0 "R47" H 5300 4250 50  0000 L CNN
 F 1 "6k8/160" H 5300 4175 50  0000 L CNN
 F 2 "Resistor_SMD:R_0603_1608Metric" H 5250 4250 50  0001 C CNN
@@
 AR Path="/63D5F044/632B472F" Ref="JP?"  Part="1"
 AR Path="/63DA5A81/632B472F" Ref="JP?"  Part="1"
-F 0 "JP1" H 5200 3630 50  0000 C CNN
+F 0 "JP7" H 5200 3630 50  0000 C CNN
 F 1 "V_SEL" H 5200 3539 50  0000 C CNN
 F 2 "Jumper:SolderJumper-3_P1.3mm_Open_RoundedPad1.0x1.5mm" H 5200 3425 50  0001 C CNN
@@
 AR Path="/63D5F044/632B4738" Ref="J?"  Part="1"
 AR Path="/63DA5A81/632B4738" Ref="J?"  Part="1"
-F 0 "J7" H 5050 3725 50  0000 L CNN
+F 0 "J15" H 5050 3725 50  0000 L CNN
 F 1 "Pressure 1" H 5050 3625 50  0000 L CNN
 F 2 "Connector_JST:JST_GH_BM04B-GHS-TBT_1x04-1MP_P1.25mm_Vertical" H 4975 3725 50  0001 C CNN
@@
 AR Path="/63D5F044/632B4751" Ref="R?"  Part="1"
 AR Path="/63DA5A81/632B4751" Ref="R?"  Part="1"
-F 0 "R23" V 6050 3825 50  0000 R CNN
+F 0 "R48" V 6050 3825 50  0000 R CNN
 F 1 "9k1" V 6200 3850 50  0000 R CNN
 F 2 "Resistor_SMD:R_0603_1608Metric" H 6125 3775 50  0001 C CNN
@@
 AR Path="/63D5F044/632B4765" Ref="C?"  Part="1"
 AR Path="/63DA5A81/632B4765" Ref="C?"  Part="1"
-F 0 "C41" H 6050 3925 50  0000 L CNN
+F 0 "C53" H 6050 3925 50  0000 L CNN
 F 1 "100n" H 6075 3825 50  0000 L CNN
 F 2 "Capacitor_SMD:C_0402_1005Metric" H 6275 3900 50  0001 C CNN

Commit message: placement almost done
Connections:
- net +12V renamed +12VA
Changed lines of the file:
@@
 $Descr A4 11693 8268
 encoding utf-8
-Sheet 10 17
+Sheet 2 18
 Title ""
 Date ""
@@
 AR Path="/63D5F044/632B46F4" Ref="#PWR?"  Part="1"
 AR Path="/63DA5A81/632B46F4" Ref="#PWR?"  Part="1"
-F 0 "#PWR0154" H 4975 3925 50  0001 C CNN
+AR Path="/6308CB6A/632B46F4" Ref="#PWR0194"  Part="1"
+F 0 "#PWR0104" H 4975 3925 50  0001 C CNN
 F 1 "GND" H 4975 4025 50  0000 C CNN
 F 2 "" H 4975 4175 50  0001 C CNN
@@
 AR Path="/63D5F044/632B46FD" Ref="U?"  Part="1"
 AR Path="/63DA5A81/632B46FD" Ref="U?"  Part="1"
-F 0 "U15" H 5775 3675 50  0000 L CNN
+AR Path="/6308CB6A/632B46FD" Ref="U1"  Part="1"
+F 0 "U9" H 5775 3675 50  0000 L CNN
 F 1 "INA180B1" H 5625 3600 50  0000 L CNN
 F 2 "Package_TO_SOT_SMD:SOT-23-5" H 5725 3825 50  0001 C CNN
@@
 AR Path="/63D5F044/632B470B" Ref="C?"  Part="1"
 AR Path="/63DA5A81/632B470B" Ref="C?"  Part="1"
-F 0 "C52" V 5825 3450 50  0000 C CNN
+AR Path="/6308CB6A/632B470B" Ref="C1"  Part="1"
+F 0 "C24" V 5825 3450 50  0000 C CNN
 F 1 "100n" V 5600 3450 50  0000 C CNN
 F 2 "Capacitor_SMD:C_0402_1005Metric" H 5725 3450 50  0001 C CNN
@@
 AR Path="/63D5F044/632B4714" Ref="#PWR?"  Part="1"
 AR Path="/63DA5A81/632B4714" Ref="#PWR?"  Part="1"
-F 0 "#PWR0155" H 5575 3850 50  0001 C CNN
+AR Path="/6308CB6A/632B4714" Ref="#PWR0195"  Part="1"
+F 0 "#PWR0105" H 5575 3850 50  0001 C CNN
 F 1 "GND" H 5575 3950 50  0000 C CNN
 F 2 "" H 5575 4100 50  0001 C CNN
@@
 AR Path="/63D5F044/632B471B" Ref="R?"  Part="1"
 AR Path="/63DA5A81/632B471B" Ref="R?"  Part="1"
-F 0 "R46" H 5300 4025 50  0000 L CNN
+AR Path="/6308CB6A/632B471B" Ref="R1"  Part="1"
+F 0 "R21" H 5300 4025 50  0000 L CNN
 F 1 "4k7/0" H 5300 3950 50  0000 L CNN
 F 2 "Resistor_SMD:R_0603_1608Metric" H 5250 4000 50  0001 C CNN
@@
 AR Path="/63D5F044/632B4721" Ref="R?"  Part="1"
 AR Path="/63DA5A81/632B4721" Ref="R?"  Part="1"
-F 0 "R47" H 5300 4250 50  0000 L CNN
+AR Path="/6308CB6A/632B4721" Ref="R2"  Part="1"
+F 0 "R22" H 5300 4250 50  0000 L CNN
 F 1 "6k8/160" H 5300 4175 50  0000 L CNN
 F 2 "Resistor_SMD:R_0603_1608Metric" H 5250 4250 50  0001 C CNN
@@
 AR Path="/63D5F044/632B4727" Ref="#PWR?"  Part="1"
 AR Path="/63DA5A81/632B4727" Ref="#PWR?"  Part="1"
-F 0 "#PWR0156" H 5250 4125 50  0001 C CNN
+AR Path="/6308CB6A/632B4727" Ref="#PWR0196"  Part="1"
+F 0 "#PWR0106" H 5250 4125 50  0001 C CNN
 F 1 "GND" H 5250 4225 50  0000 C CNN
 F 2 "" H 5250 4375 50  0001 C CNN
@@
 AR Path="/63D5F044/632B472F" Ref="JP?"  Part="1"
 AR Path="/63DA5A81/632B472F" Ref="JP?"  Part="1"
-F 0 "JP7" H 5200 3630 50  0000 C CNN
+AR Path="/6308CB6A/632B472F" Ref="JP3"  Part="1"
+F 0 "JP1" H 5200 3630 50  0000 C CNN
 F 1 "V_SEL" H 5200 3539 50  0000 C CNN
 F 2 "Jumper:SolderJumper-3_P1.3mm_Open_RoundedPad1.0x1.5mm" H 5200 3425 50  0001 C CNN
@@
 AR Path="/63D5F044/632B4738" Ref="J?"  Part="1"
 AR Path="/63DA5A81/632B4738" Ref="J?"  Part="1"
-F 0 "J15" H 5050 3725 50  0000 L CNN
+AR Path="/6308CB6A/632B4738" Ref="J23"  Part="1"
+F 0 "J7" H 5050 3725 50  0000 L CNN
 F 1 "Pressure 1" H 5050 3625 50  0000 L CNN
 F 2 "Connector_JST:JST_GH_BM04B-GHS-TBT_1x04-1MP_P1.25mm_Vertical" H 4975 3725 50  0001 C CNN
@@
 AR Path="/63D5F044/632B4744" Ref="#PWR?"  Part="1"
 AR Path="/63DA5A81/632B4744" Ref="#PWR?"  Part="1"
-F 0 "#PWR0157" H 5850 3200 50  0001 C CNN
+AR Path="/6308CB6A/632B4744" Ref="#PWR0197"  Part="1"
+F 0 "#PWR0107" H 5850 3200 50  0001 C CNN
 F 1 "GND" V 5850 3250 50  0000 C CNN
 F 2 "" H 5850 3450 50  0001 C CNN
@@
 AR Path="/63D5F044/632B4751" Ref="R?"  Part="1"
 AR Path="/63DA5A81/632B4751" Ref="R?"  Part="1"
-F 0 "R48" V 6050 3825 50  0000 R CNN
+AR Path="/6308CB6A/632B4751" Ref="R7"  Part="1"
+F 0 "R23" V 6050 3825 50  0000 R CNN
 F 1 "9k1" V 6200 3850 50  0000 R CNN
 F 2 "Resistor_SMD:R_0603_1608Metric" H 6125 3775 50  0001 C CNN
@@
 AR Path="/63D5F044/632B475B" Ref="#PWR?"  Part="1"
 AR Path="/63DA5A81/632B475B" Ref="#PWR?"  Part="1"
-F 0 "#PWR0158" H 6275 3775 50  0001 C CNN
+AR Path="/6308CB6A/632B475B" Ref="#PWR0202"  Part="1"
+F 0 "#PWR0108" H 6275 3775 50  0001 C CNN
 F 1 "GND" H 6275 3875 50  0000 C CNN
 F 2 "" H 6275 4025 50  0001 C CNN
@@
 AR Path="/63D5F044/632B4765" Ref="C?"  Part="1"
 AR Path="/63DA5A81/632B4765" Ref="C?"  Part="1"
-F 0 "C53" H 6050 3925 50  0000 L CNN
+AR Path="/6308CB6A/632B4765" Ref="C2"  Part="1"
+F 0 "C41" H 6050 3925 50  0000 L CNN
 F 1 "100n" H 6075 3825 50  0000 L CNN
 F 2 "Capacitor_SMD:C_0402_1005Metric" H 6275 3900 50  0001 C CNN
@@
 	1    6275 3900
 	-1   0    0    -1
-$EndComp
-$Comp
-L power:+12V #PWR?
-U 1 1 632B476B
-P 5400 3350
-AR Path="/632B476B" Ref="#PWR?"  Part="1"
-AR Path="/63153E68/632B476B" Ref="#PWR0109"  Part="1"
-AR Path="/63B6F693/632B476B" Ref="#PWR0135"  Part="1"
-AR Path="/63BB53C9/632B476B" Ref="#PWR0143"  Part="1"
-AR Path="/63BFB3EC/632B476B" Ref="#PWR0151"  Part="1"
-AR Path="/63C417E7/632B476B" Ref="#PWR0159"  Part="1"
-AR Path="/63D5F044/632B476B" Ref="#PWR?"  Part="1"
-AR Path="/63DA5A81/632B476B" Ref="#PWR?"  Part="1"
-F 0 "#PWR0159" H 5400 3200 50  0001 C CNN
-F 1 "+12V" H 5400 3500 50  0000 C CNN
-F 2 "" H 5400 3350 50  0001 C CNN
-F 3 "" H 5400 3350 50  0001 C CNN
-	1    5400 3350
-	1    0    0    -1
 $EndComp
 $Comp
@@
 AR Path="/63D5F044/632B4771" Ref="#PWR?"  Part="1"
 AR Path="/63DA5A81/632B4771" Ref="#PWR?"  Part="1"
-F 0 "#PWR0160" H 5575 3275 50  0001 C CNN
+AR Path="/6308CB6A/632B4771" Ref="#PWR0204"  Part="1"
+F 0 "#PWR0110" H 5575 3275 50  0001 C CNN
 F 1 "+3V3" H 5575 3575 50  0000 C CNN
 F 2 "" H 5575 3425 50  0001 C CNN
@@
 AR Path="/63D5F044/632B4777" Ref="#PWR?"  Part="1"
 AR Path="/63DA5A81/632B4777" Ref="#PWR?"  Part="1"
-F 0 "#PWR0161" H 5000 3200 50  0001 C CNN
+AR Path="/6308CB6A/632B4777" Ref="#PWR0205"  Part="1"
+F 0 "#PWR0111" H 5000 3200 50  0001 C CNN
 F 1 "+5V" H 5000 3500 50  0000 C CNN
 F 2 "" H 5000 3350 50  0001 C CNN
@@
 	1    0    0    -1
 $EndComp
+$Comp
+L power:+12VA #PWR0151
+U 1 1 637AE5AB
+P 5400 3350
+AR Path="/63153E68/637AE5AB" Ref="#PWR0151"  Part="1"
+AR Path="/63B6F693/637AE5AB" Ref="#PWR0159"  Part="1"
+AR Path="/63BB53C9/637AE5AB" Ref="#PWR0203"  Part="1"
+AR Path="/63BFB3EC/637AE5AB" Ref="#PWR0212"  Part="1"
+AR Path="/63C417E7/637AE5AB" Ref="#PWR0213"  Part="1"
+AR Path="/6308CB6A/637AE5AB" Ref="#PWR0214"  Part="1"
+F 0 "#PWR0151" H 5400 3200 50  0001 C CNN
+F 1 "+12VA" H 5415 3523 50  0000 C CNN
+F 2 "" H 5400 3350 50  0001 C CNN
+F 3 "" H 5400 3350 50  0001 C CNN
+	1    5400 3350
+	1    0    0    -1
+$EndComp

Commit message: fixed net names
Parts:
- J7: value Pressure 1 -> Pressure
Changed lines of the file:
@@
 $Descr A4 11693 8268
 encoding utf-8
-Sheet 2 18
+Sheet 18 18
 Title ""
 Date ""
@@
 AR Path="/63DA5A81/632B46F4" Ref="#PWR?"  Part="1"
 AR Path="/6308CB6A/632B46F4" Ref="#PWR0194"  Part="1"
-F 0 "#PWR0104" H 4975 3925 50  0001 C CNN
+F 0 "#PWR0194" H 4975 3925 50  0001 C CNN
 F 1 "GND" H 4975 4025 50  0000 C CNN
 F 2 "" H 4975 4175 50  0001 C CNN
@@
 AR Path="/63DA5A81/632B46FD" Ref="U?"  Part="1"
 AR Path="/6308CB6A/632B46FD" Ref="U1"  Part="1"
-F 0 "U9" H 5775 3675 50  0000 L CNN
+F 0 "U1" H 5775 3675 50  0000 L CNN
 F 1 "INA180B1" H 5625 3600 50  0000 L CNN
 F 2 "Package_TO_SOT_SMD:SOT-23-5" H 5725 3825 50  0001 C CNN
@@
 AR Path="/63DA5A81/632B470B" Ref="C?"  Part="1"
 AR Path="/6308CB6A/632B470B" Ref="C1"  Part="1"
-F 0 "C24" V 5825 3450 50  0000 C CNN
+F 0 "C1" V 5825 3450 50  0000 C CNN
 F 1 "100n" V 5600 3450 50  0000 C CNN
 F 2 "Capacitor_SMD:C_0402_1005Metric" H 5725 3450 50  0001 C CNN
@@
 AR Path="/63DA5A81/632B4714" Ref="#PWR?"  Part="1"
 AR Path="/6308CB6A/632B4714" Ref="#PWR0195"  Part="1"
-F 0 "#PWR0105" H 5575 3850 50  0001 C CNN
+F 0 "#PWR0195" H 5575 3850 50  0001 C CNN
 F 1 "GND" H 5575 3950 50  0000 C CNN
 F 2 "" H 5575 4100 50  0001 C CNN
@@
 AR Path="/63DA5A81/632B471B" Ref="R?"  Part="1"
 AR Path="/6308CB6A/632B471B" Ref="R1"  Part="1"
-F 0 "R21" H 5300 4025 50  0000 L CNN
+F 0 "R1" H 5300 4025 50  0000 L CNN
 F 1 "4k7/0" H 5300 3950 50  0000 L CNN
 F 2 "Resistor_SMD:R_0603_1608Metric" H 5250 4000 50  0001 C CNN
@@
 AR Path="/63DA5A81/632B4721" Ref="R?"  Part="1"
 AR Path="/6308CB6A/632B4721" Ref="R2"  Part="1"
-F 0 "R22" H 5300 4250 50  0000 L CNN
+F 0 "R2" H 5300 4250 50  0000 L CNN
 F 1 "6k8/160" H 5300 4175 50  0000 L CNN
 F 2 "Resistor_SMD:R_0603_1608Metric" H 5250 4250 50  0001 C CNN
@@
 AR Path="/63DA5A81/632B4727" Ref="#PWR?"  Part="1"
 AR Path="/6308CB6A/632B4727" Ref="#PWR0196"  Part="1"
-F 0 "#PWR0106" H 5250 4125 50  0001 C CNN
+F 0 "#PWR0196" H 5250 4125 50  0001 C CNN
 F 1 "GND" H 5250 4225 50  0000 C CNN
 F 2 "" H 5250 4375 50  0001 C CNN
@@
 AR Path="/63DA5A81/632B472F" Ref="JP?"  Part="1"
 AR Path="/6308CB6A/632B472F" Ref="JP3"  Part="1"
-F 0 "JP1" H 5200 3630 50  0000 C CNN
+F 0 "JP3" H 5200 3630 50  0000 C CNN
 F 1 "V_SEL" H 5200 3539 50  0000 C CNN
 F 2 "Jumper:SolderJumper-3_P1.3mm_Open_RoundedPad1.0x1.5mm" H 5200 3425 50  0001 C CNN
@@
 AR Path="/63DA5A81/632B4738" Ref="J?"  Part="1"
 AR Path="/6308CB6A/632B4738" Ref="J23"  Part="1"
-F 0 "J7" H 5050 3725 50  0000 L CNN
-F 1 "Pressure 1" H 5050 3625 50  0000 L CNN
+F 0 "J23" H 5050 3725 50  0000 L CNN
+F 1 "Pressure" H 5050 3625 50  0000 L CNN
 F 2 "Connector_JST:JST_GH_BM04B-GHS-TBT_1x04-1MP_P1.25mm_Vertical" H 4975 3725 50  0001 C CNN
 F 3 "~" H 4975 3725 50  0001 C CNN
@@
 AR Path="/63DA5A81/632B4744" Ref="#PWR?"  Part="1"
 AR Path="/6308CB6A/632B4744" Ref="#PWR0197"  Part="1"
-F 0 "#PWR0107" H 5850 3200 50  0001 C CNN
+F 0 "#PWR0197" H 5850 3200 50  0001 C CNN
 F 1 "GND" V 5850 3250 50  0000 C CNN
 F 2 "" H 5850 3450 50  0001 C CNN
@@
 AR Path="/63DA5A81/632B4751" Ref="R?"  Part="1"
 AR Path="/6308CB6A/632B4751" Ref="R7"  Part="1"
-F 0 "R23" V 6050 3825 50  0000 R CNN
+F 0 "R7" V 6050 3825 50  0000 R CNN
 F 1 "9k1" V 6200 3850 50  0000 R CNN
 F 2 "Resistor_SMD:R_0603_1608Metric" H 6125 3775 50  0001 C CNN
@@
 AR Path="/63DA5A81/632B475B" Ref="#PWR?"  Part="1"
 AR Path="/6308CB6A/632B475B" Ref="#PWR0202"  Part="1"
-F 0 "#PWR0108" H 6275 3775 50  0001 C CNN
+F 0 "#PWR0202" H 6275 3775 50  0001 C CNN
 F 1 "GND" H 6275 3875 50  0000 C CNN
 F 2 "" H 6275 4025 50  0001 C CNN
@@
 AR Path="/63DA5A81/632B4765" Ref="C?"  Part="1"
 AR Path="/6308CB6A/632B4765" Ref="C2"  Part="1"
-F 0 "C41" H 6050 3925 50  0000 L CNN
+F 0 "C2" H 6050 3925 50  0000 L CNN
 F 1 "100n" H 6075 3825 50  0000 L CNN
 F 2 "Capacitor_SMD:C_0402_1005Metric" H 6275 3900 50  0001 C CNN
@@
 AR Path="/63DA5A81/632B4771" Ref="#PWR?"  Part="1"
 AR Path="/6308CB6A/632B4771" Ref="#PWR0204"  Part="1"
-F 0 "#PWR0110" H 5575 3275 50  0001 C CNN
+F 0 "#PWR0204" H 5575 3275 50  0001 C CNN
 F 1 "+3V3" H 5575 3575 50  0000 C CNN
 F 2 "" H 5575 3425 50  0001 C CNN
@@
 AR Path="/63DA5A81/632B4777" Ref="#PWR?"  Part="1"
 AR Path="/6308CB6A/632B4777" Ref="#PWR0205"  Part="1"
-F 0 "#PWR0111" H 5000 3200 50  0001 C CNN
+F 0 "#PWR0205" H 5000 3200 50  0001 C CNN
 F 1 "+5V" H 5000 3500 50  0000 C CNN
 F 2 "" H 5000 3350 50  0001 C CNN
@@
 AR Path="/63C417E7/637AE5AB" Ref="#PWR0213"  Part="1"
 AR Path="/6308CB6A/637AE5AB" Ref="#PWR0214"  Part="1"
-F 0 "#PWR0151" H 5400 3200 50  0001 C CNN
+F 0 "#PWR0214" H 5400 3200 50  0001 C CNN
 F 1 "+12VA" H 5415 3523 50  0000 C CNN
 F 2 "" H 5400 3350 50  0001 C CNN

Commit message: small improvements, updated doc
Changed lines of the file:
@@
 $Descr A4 11693 8268
 encoding utf-8
-Sheet 16 18
+Sheet 2 18
 Title ""
 Date ""
@@
 AR Path="/63DA5A81/632B46F4" Ref="#PWR?"  Part="1"
 AR Path="/6308CB6A/632B46F4" Ref="#PWR0194"  Part="1"
-F 0 "#PWR0194" H 4975 3925 50  0001 C CNN
+F 0 "#PWR0104" H 4975 3925 50  0001 C CNN
 F 1 "GND" H 4975 4025 50  0000 C CNN
 F 2 "" H 4975 4175 50  0001 C CNN
@@
 AR Path="/63DA5A81/632B46FD" Ref="U?"  Part="1"
 AR Path="/6308CB6A/632B46FD" Ref="U1"  Part="1"
-F 0 "U1" H 5775 3675 50  0000 L CNN
+F 0 "U9" H 5775 3675 50  0000 L CNN
 F 1 "INA180B1" H 5625 3600 50  0000 L CNN
 F 2 "Package_TO_SOT_SMD:SOT-23-5" H 5725 3825 50  0001 C CNN
@@
 AR Path="/63DA5A81/632B470B" Ref="C?"  Part="1"
 AR Path="/6308CB6A/632B470B" Ref="C1"  Part="1"
-F 0 "C1" V 5825 3450 50  0000 C CNN
+F 0 "C24" V 5825 3450 50  0000 C CNN
 F 1 "100n" V 5600 3450 50  0000 C CNN
 F 2 "Capacitor_SMD:C_0402_1005Metric" H 5725 3450 50  0001 C CNN
@@
 AR Path="/63DA5A81/632B4714" Ref="#PWR?"  Part="1"
 AR Path="/6308CB6A/632B4714" Ref="#PWR0195"  Part="1"
-F 0 "#PWR0195" H 5575 3850 50  0001 C CNN
+F 0 "#PWR0105" H 5575 3850 50  0001 C CNN
 F 1 "GND" H 5575 3950 50  0000 C CNN
 F 2 "" H 5575 4100 50  0001 C CNN
@@
 AR Path="/63DA5A81/632B471B" Ref="R?"  Part="1"
 AR Path="/6308CB6A/632B471B" Ref="R1"  Part="1"
-F 0 "R1" H 5300 4025 50  0000 L CNN
+F 0 "R21" H 5300 4025 50  0000 L CNN
 F 1 "4k7/0" H 5300 3950 50  0000 L CNN
 F 2 "Resistor_SMD:R_0603_1608Metric" H 5250 4000 50  0001 C CNN
@@
 AR Path="/63DA5A81/632B4721" Ref="R?"  Part="1"
 AR Path="/6308CB6A/632B4721" Ref="R2"  Part="1"
-F 0 "R2" H 5300 4250 50  0000 L CNN
+F 0 "R22" H 5300 4250 50  0000 L CNN
 F 1 "6k8/160" H 5300 4175 50  0000 L CNN
 F 2 "Resistor_SMD:R_0603_1608Metric" H 5250 4250 50  0001 C CNN
@@
 AR Path="/63DA5A81/632B4727" Ref="#PWR?"  Part="1"
 AR Path="/6308CB6A/632B4727" Ref="#PWR0196"  Part="1"
-F 0 "#PWR0196" H 5250 4125 50  0001 C CNN
+F 0 "#PWR0106" H 5250 4125 50  0001 C CNN
 F 1 "GND" H 5250 4225 50  0000 C CNN
 F 2 "" H 5250 4375 50  0001 C CNN
@@
 AR Path="/63DA5A81/632B472F" Ref="JP?"  Part="1"
 AR Path="/6308CB6A/632B472F" Ref="JP3"  Part="1"
-F 0 "JP3" H 5200 3630 50  0000 C CNN
+F 0 "JP1" H 5200 3630 50  0000 C CNN
 F 1 "V_SEL" H 5200 3539 50  0000 C CNN
 F 2 "Jumper:SolderJumper-3_P1.3mm_Open_RoundedPad1.0x1.5mm" H 5200 3425 50  0001 C CNN
@@
 AR Path="/63DA5A81/632B4738" Ref="J?"  Part="1"
 AR Path="/6308CB6A/632B4738" Ref="J23"  Part="1"
-F 0 "J23" H 5050 3725 50  0000 L CNN
+F 0 "J7" H 5050 3725 50  0000 L CNN
 F 1 "Pressure" H 5050 3625 50  0000 L CNN
 F 2 "Connector_JST:JST_GH_BM04B-GHS-TBT_1x04-1MP_P1.25mm_Vertical" H 4975 3725 50  0001 C CNN
@@
 AR Path="/63DA5A81/632B4744" Ref="#PWR?"  Part="1"
 AR Path="/6308CB6A/632B4744" Ref="#PWR0197"  Part="1"
-F 0 "#PWR0197" H 5850 3200 50  0001 C CNN
+F 0 "#PWR0107" H 5850 3200 50  0001 C CNN
 F 1 "GND" V 5850 3250 50  0000 C CNN
 F 2 "" H 5850 3450 50  0001 C CNN
@@
 AR Path="/63DA5A81/632B4751" Ref="R?"  Part="1"
 AR Path="/6308CB6A/632B4751" Ref="R7"  Part="1"
-F 0 "R7" V 6050 3825 50  0000 R CNN
+F 0 "R23" V 6050 3825 50  0000 R CNN
 F 1 "9k1" V 6200 3850 50  0000 R CNN
 F 2 "Resistor_SMD:R_0603_1608Metric" H 6125 3775 50  0001 C CNN
@@
 AR Path="/63DA5A81/632B475B" Ref="#PWR?"  Part="1"
 AR Path="/6308CB6A/632B475B" Ref="#PWR0202"  Part="1"
-F 0 "#PWR0202" H 6275 3775 50  0001 C CNN
+F 0 "#PWR0108" H 6275 3775 50  0001 C CNN
 F 1 "GND" H 6275 3875 50  0000 C CNN
 F 2 "" H 6275 4025 50  0001 C CNN
@@
 AR Path="/63DA5A81/632B4765" Ref="C?"  Part="1"
 AR Path="/6308CB6A/632B4765" Ref="C2"  Part="1"
-F 0 "C2" H 6050 3925 50  0000 L CNN
+F 0 "C41" H 6050 3925 50  0000 L CNN
 F 1 "100n" H 6075 3825 50  0000 L CNN
 F 2 "Capacitor_SMD:C_0402_1005Metric" H 6275 3900 50  0001 C CNN
@@
 AR Path="/63DA5A81/632B4771" Ref="#PWR?"  Part="1"
 AR Path="/6308CB6A/632B4771" Ref="#PWR0204"  Part="1"
-F 0 "#PWR0204" H 5575 3275 50  0001 C CNN
+F 0 "#PWR0110" H 5575 3275 50  0001 C CNN
 F 1 "+3V3" H 5575 3575 50  0000 C CNN
 F 2 "" H 5575 3425 50  0001 C CNN
@@
 AR Path="/63DA5A81/632B4777" Ref="#PWR?"  Part="1"
 AR Path="/6308CB6A/632B4777" Ref="#PWR0205"  Part="1"
-F 0 "#PWR0205" H 5000 3200 50  0001 C CNN
+F 0 "#PWR0111" H 5000 3200 50  0001 C CNN
 F 1 "+5V" H 5000 3500 50  0000 C CNN
 F 2 "" H 5000 3350 50  0001 C CNN
@@
 AR Path="/63C417E7/637AE5AB" Ref="#PWR0213"  Part="1"
 AR Path="/6308CB6A/637AE5AB" Ref="#PWR0214"  Part="1"
-F 0 "#PWR0214" H 5400 3200 50  0001 C CNN
+F 0 "#PWR0151" H 5400 3200 50  0001 C CNN
 F 1 "+12VA" H 5415 3523 50  0000 C CNN
 F 2 "" H 5400 3350 50  0001 C CNN
