File: PressureSensorInput.sch (KiCad schematic (older format))
At the start: 8 parts, among them J7 Pressure, U9 INA180B1

Commit message: some more small changes
Parts:
- R21: value 4k7/0 -> 5k6/0
- R22: value 6k8/160 -> 10k/160
- R23: value 9k1 -> 10k
Other:
- note added: "op-amp for diff. 150mV bridge input,\nvoltage div. for 0-5V or 4-20mA input.\n(5k6/10k for 0-5V, 0/160R for 4-20mA)"
- note removed: "op-amp for diff. 150mV bridge input,\nvoltage div. for 0-5V or 4-20mA input.\n(4.7k/6.8k for 0-5V,\n0/160 Ohm for 4-20mA)"
Changed lines of the file:
@@
 AR Path="/63DA5A81/632B46F4" Ref="#PWR?"  Part="1"
 AR Path="/6308CB6A/632B46F4" Ref="#PWR0194"  Part="1"
-F 0 "#PWR0104" H 4975 3925 50  0001 C CNN
+F 0 "#PWR0194" H 4975 3925 50  0001 C CNN
 F 1 "GND" H 4975 4025 50  0000 C CNN
 F 2 "" H 4975 4175 50  0001 C CNN
@@
 AR Path="/63DA5A81/632B4714" Ref="#PWR?"  Part="1"
 AR Path="/6308CB6A/632B4714" Ref="#PWR0195"  Part="1"
-F 0 "#PWR0105" H 5575 3850 50  0001 C CNN
+F 0 "#PWR0195" H 5575 3850 50  0001 C CNN
 F 1 "GND" H 5575 3950 50  0000 C CNN
 F 2 "" H 5575 4100 50  0001 C CNN
@@
 AR Path="/6308CB6A/632B471B" Ref="R1"  Part="1"
 F 0 "R21" H 5300 4025 50  0000 L CNN
-F 1 "4k7/0" H 5300 3950 50  0000 L CNN
+F 1 "5k6/0" H 5300 3950 50  0000 L CNN
 F 2 "Resistor_SMD:R_0603_1608Metric" H 5250 4000 50  0001 C CNN
 F 3 "~" H 5250 4000 50  0001 C CNN
@@
 AR Path="/6308CB6A/632B4721" Ref="R2"  Part="1"
 F 0 "R22" H 5300 4250 50  0000 L CNN
-F 1 "6k8/160" H 5300 4175 50  0000 L CNN
+F 1 "10k/160" H 5300 4175 50  0000 L CNN
 F 2 "Resistor_SMD:R_0603_1608Metric" H 5250 4250 50  0001 C CNN
 F 3 "~" H 5250 4250 50  0001 C CNN
@@
 AR Path="/63DA5A81/632B4727" Ref="#PWR?"  Part="1"
 AR Path="/6308CB6A/632B4727" Ref="#PWR0196"  Part="1"
-F 0 "#PWR0106" H 5250 4125 50  0001 C CNN
+F 0 "#PWR0196" H 5250 4125 50  0001 C CNN
 F 1 "GND" H 5250 4225 50  0000 C CNN
 F 2 "" H 5250 4375 50  0001 C CNN
@@
 	5250 4375 5250 4350
 Text Notes 5675 4525 0    50   ~ 0
-op-amp for diff. 150mV bridge input,\nvoltage div. for 0-5V or 4-20mA input.\n(4.7k/6.8k for 0-5V,\n0/160 Ohm for 4-20mA)
+op-amp for diff. 150mV bridge input,\nvoltage div. for 0-5V or 4-20mA input.\n(5k6/10k for 0-5V, 0/160R for 4-20mA)
 $Comp
 L Jumper:SolderJumper_3_Open JP?
@@
 AR Path="/63DA5A81/632B4744" Ref="#PWR?"  Part="1"
 AR Path="/6308CB6A/632B4744" Ref="#PWR0197"  Part="1"
-F 0 "#PWR0107" H 5850 3200 50  0001 C CNN
+F 0 "#PWR0197" H 5850 3200 50  0001 C CNN
 F 1 "GND" V 5850 3250 50  0000 C CNN
 F 2 "" H 5850 3450 50  0001 C CNN
@@
 AR Path="/6308CB6A/632B4751" Ref="R7"  Part="1"
 F 0 "R23" V 6050 3825 50  0000 R CNN
-F 1 "9k1" V 6200 3850 50  0000 R CNN
+F 1 "10k" V 6200 3850 50  0000 R CNN
 F 2 "Resistor_SMD:R_0603_1608Metric" H 6125 3775 50  0001 C CNN
 F 3 "~" H 6125 3775 50  0001 C CNN
@@
 AR Path="/63DA5A81/632B475B" Ref="#PWR?"  Part="1"
 AR Path="/6308CB6A/632B475B" Ref="#PWR0202"  Part="1"
-F 0 "#PWR0108" H 6275 3775 50  0001 C CNN
+F 0 "#PWR0202" H 6275 3775 50  0001 C CNN
 F 1 "GND" H 6275 3875 50  0000 C CNN
 F 2 "" H 6275 4025 50  0001 C CNN
@@
 AR Path="/63DA5A81/632B4771" Ref="#PWR?"  Part="1"
 AR Path="/6308CB6A/632B4771" Ref="#PWR0204"  Part="1"
-F 0 "#PWR0110" H 5575 3275 50  0001 C CNN
+F 0 "#PWR0204" H 5575 3275 50  0001 C CNN
 F 1 "+3V3" H 5575 3575 50  0000 C CNN
 F 2 "" H 5575 3425 50  0001 C CNN
@@
 AR Path="/63DA5A81/632B4777" Ref="#PWR?"  Part="1"
 AR Path="/6308CB6A/632B4777" Ref="#PWR0205"  Part="1"
-F 0 "#PWR0111" H 5000 3200 50  0001 C CNN
+F 0 "#PWR0205" H 5000 3200 50  0001 C CNN
 F 1 "+5V" H 5000 3500 50  0000 C CNN
 F 2 "" H 5000 3350 50  0001 C CNN
@@
 AR Path="/63C417E7/637AE5AB" Ref="#PWR0213"  Part="1"
 AR Path="/6308CB6A/637AE5AB" Ref="#PWR0214"  Part="1"
-F 0 "#PWR0151" H 5400 3200 50  0001 C CNN
+F 0 "#PWR0214" H 5400 3200 50  0001 C CNN
 F 1 "+12VA" H 5415 3523 50  0000 C CNN
 F 2 "" H 5400 3350 50  0001 C CNN
