File: ServoOutput.sch (KiCad schematic (older format))
At the start: 7 parts, among them J9 Servo 1, U10 INA180B1

Commit message: preliminary placement done
Parts:
- J9: footprint Connector_Molex:Molex_Nano-Fit_105313-xx04_1x04_P2.50mm_Horizontal -> TXV_LIB:Molex_Nano-Fit_105313-xx04_1x04_P2.50mm_Horizontal
Changed lines of the file:
@@
 F 0 "J18" H 6300 3625 50  0000 C CNN
 F 1 "Servo 1" H 6300 3550 50  0000 C CNN
-F 2 "Connector_Molex:Molex_Nano-Fit_105313-xx04_1x04_P2.50mm_Horizontal" H 6300 3350 50  0001 C CNN
+F 2 "TXV_LIB:Molex_Nano-Fit_105313-xx04_1x04_P2.50mm_Horizontal" H 6300 3350 50  0001 C CNN
 F 3 "~" H 6300 3350 50  0001 C CNN
 	1    6300 3350
@@
 AR Path="/63F9E75F/63587B22" Ref="#PWR0166"  Part="1"
 AR Path="/63FE6097/63587B22" Ref="#PWR0171"  Part="1"
-F 0 "#PWR0171" H 6300 3575 50  0001 C CNN
+F 0 "#PWR0166" H 6300 3575 50  0001 C CNN
 F 1 "GND" H 6300 3675 50  0000 C CNN
 F 2 "" H 6300 3825 50  0001 C CNN
@@
 AR Path="/63F9E75F/63587B2C" Ref="#PWR0167"  Part="1"
 AR Path="/63FE6097/63587B2C" Ref="#PWR0172"  Part="1"
-F 0 "#PWR0172" H 5225 3525 50  0001 C CNN
+F 0 "#PWR0167" H 5225 3525 50  0001 C CNN
 F 1 "GND" H 5225 3625 50  0000 C CNN
 F 2 "" H 5225 3775 50  0001 C CNN
@@
 AR Path="/63F9E75F/63587B5F" Ref="#PWR0168"  Part="1"
 AR Path="/63FE6097/63587B5F" Ref="#PWR0173"  Part="1"
-F 0 "#PWR0173" H 5425 3750 50  0001 C CNN
+F 0 "#PWR0168" H 5425 3750 50  0001 C CNN
 F 1 "+3V3" H 5425 4050 50  0000 C CNN
 F 2 "" H 5425 3900 50  0001 C CNN
@@
 AR Path="/63F9E75F/63587B6D" Ref="#PWR0169"  Part="1"
 AR Path="/63FE6097/63587B6D" Ref="#PWR0174"  Part="1"
-F 0 "#PWR0174" H 5500 3925 50  0001 C CNN
+F 0 "#PWR0169" H 5500 3925 50  0001 C CNN
 F 1 "GND" H 5500 4025 50  0000 C CNN
 F 2 "" H 5500 4175 50  0001 C CNN
@@
 AR Path="/63F9E75F/63587B8A" Ref="#PWR0170"  Part="1"
 AR Path="/63FE6097/63587B8A" Ref="#PWR0175"  Part="1"
-F 0 "#PWR0175" H 5650 3500 50  0001 C CNN
+F 0 "#PWR0170" H 5650 3500 50  0001 C CNN
 F 1 "+7.4V" V 5650 3750 50  0000 L CNN
 F 2 "" H 5650 3650 50  0001 C CNN

Commit message: changed form factor to better fit into uHb engine section
Parts:
- J9: footprint TXV_LIB:Molex_Nano-Fit_105313-xx04_1x04_P2.50mm_Horizontal -> TXV_LIB:Molex_Nano-Fit_105309-xx04_1x04_P2.50mm_Vertical
Changed lines of the file:
@@
 $Descr A4 11693 8268
 encoding utf-8
-Sheet 13 17
+Sheet 4 17
 Title ""
 Date ""
@@
 AR Path="/63F9E75F/63587B1C" Ref="J18"  Part="1"
 AR Path="/63FE6097/63587B1C" Ref="J19"  Part="1"
-F 0 "J18" H 6300 3625 50  0000 C CNN
+F 0 "J9" H 6300 3625 50  0000 C CNN
 F 1 "Servo 1" H 6300 3550 50  0000 C CNN
-F 2 "TXV_LIB:Molex_Nano-Fit_105313-xx04_1x04_P2.50mm_Horizontal" H 6300 3350 50  0001 C CNN
+F 2 "TXV_LIB:Molex_Nano-Fit_105309-xx04_1x04_P2.50mm_Vertical" H 6300 3350 50  0001 C CNN
 F 3 "~" H 6300 3350 50  0001 C CNN
 	1    6300 3350
@@
 AR Path="/63F9E75F/63587B22" Ref="#PWR0166"  Part="1"
 AR Path="/63FE6097/63587B22" Ref="#PWR0171"  Part="1"
-F 0 "#PWR0166" H 6300 3575 50  0001 C CNN
+F 0 "#PWR0114" H 6300 3575 50  0001 C CNN
 F 1 "GND" H 6300 3675 50  0000 C CNN
 F 2 "" H 6300 3825 50  0001 C CNN
@@
 AR Path="/63F9E75F/63587B2C" Ref="#PWR0167"  Part="1"
 AR Path="/63FE6097/63587B2C" Ref="#PWR0172"  Part="1"
-F 0 "#PWR0167" H 5225 3525 50  0001 C CNN
+F 0 "#PWR0115" H 5225 3525 50  0001 C CNN
 F 1 "GND" H 5225 3625 50  0000 C CNN
 F 2 "" H 5225 3775 50  0001 C CNN
@@
 AR Path="/63F9E75F/63587B33" Ref="R51"  Part="1"
 AR Path="/63FE6097/63587B33" Ref="R54"  Part="1"
-F 0 "R51" H 5166 3354 50  0000 R CNN
+F 0 "R25" H 5166 3354 50  0000 R CNN
 F 1 "9k1" H 5166 3445 50  0000 R CNN
 F 2 "Resistor_SMD:R_0603_1608Metric" H 5225 3400 50  0001 C CNN
@@
 AR Path="/63F9E75F/63587B41" Ref="R52"  Part="1"
 AR Path="/63FE6097/63587B41" Ref="R55"  Part="1"
-F 0 "R52" V 5750 3575 50  0000 L CNN
+F 0 "R26" V 5750 3575 50  0000 L CNN
 F 1 "10m 1W" V 5900 3475 50  0000 L CNN
 F 2 "Resistor_SMD:R_1206_3216Metric" H 5825 3650 50  0001 C CNN
@@
 AR Path="/63F9E75F/63587B47" Ref="R53"  Part="1"
 AR Path="/63FE6097/63587B47" Ref="R56"  Part="1"
-F 0 "R53" V 6000 3575 50  0000 R CNN
+F 0 "R27" V 6000 3575 50  0000 R CNN
 F 1 "1k" V 6025 3425 50  0000 R CNN
 F 2 "Resistor_SMD:R_0603_1608Metric" H 5950 3350 50  0001 C CNN
@@
 AR Path="/63F9E75F/63587B4F" Ref="C56"  Part="1"
 AR Path="/63FE6097/63587B4F" Ref="C58"  Part="1"
-F 0 "C56" H 5025 3675 50  0000 L CNN
+F 0 "C43" H 5025 3675 50  0000 L CNN
 F 1 "100n" H 5025 3575 50  0000 L CNN
 F 2 "Capacitor_SMD:C_0402_1005Metric" H 5225 3650 50  0001 C CNN
@@
 AR Path="/63F9E75F/63587B59" Ref="U16"  Part="1"
 AR Path="/63FE6097/63587B59" Ref="U17"  Part="1"
-F 0 "U16" V 5825 3750 50  0000 L CNN
+F 0 "U10" V 5825 3750 50  0000 L CNN
 F 1 "INA180B1" V 5925 3575 50  0000 L CNN
 F 2 "Package_TO_SOT_SMD:SOT-23-5" H 5875 4075 50  0001 C CNN
@@
 AR Path="/63F9E75F/63587B5F" Ref="#PWR0168"  Part="1"
 AR Path="/63FE6097/63587B5F" Ref="#PWR0173"  Part="1"
-F 0 "#PWR0168" H 5425 3750 50  0001 C CNN
+F 0 "#PWR0116" H 5425 3750 50  0001 C CNN
 F 1 "+3V3" H 5425 4050 50  0000 C CNN
 F 2 "" H 5425 3900 50  0001 C CNN
@@
 AR Path="/63F9E75F/63587B66" Ref="C57"  Part="1"
 AR Path="/63FE6097/63587B66" Ref="C59"  Part="1"
-F 0 "C57" H 5425 4125 50  0000 C CNN
+F 0 "C44" H 5425 4125 50  0000 C CNN
 F 1 "100n" H 5375 3975 50  0000 C CNN
 F 2 "Capacitor_SMD:C_0402_1005Metric" H 5500 4050 50  0001 C CNN
@@
 AR Path="/63F9E75F/63587B6D" Ref="#PWR0169"  Part="1"
 AR Path="/63FE6097/63587B6D" Ref="#PWR0174"  Part="1"
-F 0 "#PWR0169" H 5500 3925 50  0001 C CNN
+F 0 "#PWR0117" H 5500 3925 50  0001 C CNN
 F 1 "GND" H 5500 4025 50  0000 C CNN
 F 2 "" H 5500 4175 50  0001 C CNN
@@
 AR Path="/63F9E75F/63587B8A" Ref="#PWR0170"  Part="1"
 AR Path="/63FE6097/63587B8A" Ref="#PWR0175"  Part="1"
-F 0 "#PWR0170" H 5650 3500 50  0001 C CNN
+F 0 "#PWR0118" H 5650 3500 50  0001 C CNN
 F 1 "+7.4V" V 5650 3750 50  0000 L CNN
 F 2 "" H 5650 3650 50  0001 C CNN

Commit message: placement almost done
Parts:
- added D14: OUT 1, LED_SMD:LED_0603_1608Metric, symbol Device:LED_Small_ALT
- added R10: 120, Resistor_SMD:R_0603_1608Metric, symbol Device:R_Small
Connections:
- net labels added: LED, VS
- net labels removed: +7.4V
- wire segments 33 -> 37
Changed lines of the file:
@@
 $Descr A4 11693 8268
 encoding utf-8
-Sheet 4 17
+Sheet 4 18
 Title ""
 Date ""
@@
 	5425 3925 5500 3925
 Connection ~ 5500 3925
-$Comp
-L TXV_LIB:+7.4V #PWR?
-U 1 1 63587B8A
-P 5650 3650
-AR Path="/63587B8A" Ref="#PWR?"  Part="1"
-AR Path="/634CE57C/63587B8A" Ref="#PWR0118"  Part="1"
-AR Path="/63F9E75F/63587B8A" Ref="#PWR0170"  Part="1"
-AR Path="/63FE6097/63587B8A" Ref="#PWR0175"  Part="1"
-F 0 "#PWR0118" H 5650 3500 50  0001 C CNN
-F 1 "+7.4V" V 5650 3750 50  0000 L CNN
-F 2 "" H 5650 3650 50  0001 C CNN
-F 3 "" H 5650 3650 50  0001 C CNN
-	1    5650 3650
-	0    -1   -1   0
-$EndComp
 Text Notes 5900 4250 0    50   ~ 0
 (Gain 20)
@@
 Text HLabel 6000 4350 2    50   Output ~ 0
 Current
+$Comp
+L power:VS #PWR0118
+U 1 1 62FB5B89
+P 5650 3650
+AR Path="/634CE57C/62FB5B89" Ref="#PWR0118"  Part="1"
+AR Path="/63F9E75F/62FB5B89" Ref="#PWR0170"  Part="1"
+AR Path="/63FE6097/62FB5B89" Ref="#PWR0175"  Part="1"
+F 0 "#PWR0118" H 5450 3500 50  0001 C CNN
+F 1 "VS" V 5650 3775 50  0000 L CNN
+F 2 "" H 5650 3650 50  0001 C CNN
+F 3 "" H 5650 3650 50  0001 C CNN
+	1    5650 3650
+	0    -1   -1   0
+$EndComp
+$Comp
+L Device:LED_Small_ALT D?
+U 1 1 632B8B39
+P 4800 3925
+AR Path="/632B8B39" Ref="D?"  Part="1"
+AR Path="/636FF559/632B8B39" Ref="D?"  Part="1"
+AR Path="/64079439/632B8B39" Ref="D?"  Part="1"
+AR Path="/634CE57C/632B8B39" Ref="D14"  Part="1"
+AR Path="/63F9E75F/632B8B39" Ref="D15"  Part="1"
+AR Path="/63FE6097/632B8B39" Ref="D16"  Part="1"
+F 0 "D14" V 4825 4125 50  0000 R CNN
+F 1 "OUT 1" V 4750 4225 50  0000 R CNN
+F 2 "LED_SMD:LED_0603_1608Metric" V 4800 3925 50  0001 C CNN
+F 3 "~" V 4800 3925 50  0001 C CNN
+	1    4800 3925
+	0    -1   -1   0
+$EndComp
+$Comp
+L power:GND #PWR?
+U 1 1 632B8B3F
+P 4800 4050
+AR Path="/632B8B3F" Ref="#PWR?"  Part="1"
+AR Path="/636FF559/632B8B3F" Ref="#PWR?"  Part="1"
+AR Path="/64079439/632B8B3F" Ref="#PWR?"  Part="1"
+AR Path="/634CE57C/632B8B3F" Ref="#PWR0209"  Part="1"
+AR Path="/63F9E75F/632B8B3F" Ref="#PWR0210"  Part="1"
+AR Path="/63FE6097/632B8B3F" Ref="#PWR0211"  Part="1"
+F 0 "#PWR0209" H 4800 3800 50  0001 C CNN
+F 1 "GND" H 4800 3900 50  0000 C CNN
+F 2 "" H 4800 4050 50  0001 C CNN
+F 3 "" H 4800 4050 50  0001 C CNN
+	1    4800 4050
+	1    0    0    -1
+$EndComp
+Wire Wire Line
+	4800 4050 4800 4025
+Wire Wire Line
+	4800 3800 4800 3825
+$Comp
+L Device:R_Small R?
+U 1 1 632B8B47
+P 4800 3700
+AR Path="/6015C35D/632B8B47" Ref="R?"  Part="1"
+AR Path="/632B8B47" Ref="R?"  Part="1"
+AR Path="/636FF559/632B8B47" Ref="R?"  Part="1"
+AR Path="/64079439/632B8B47" Ref="R?"  Part="1"
+AR Path="/634CE57C/632B8B47" Ref="R10"  Part="1"
+AR Path="/63F9E75F/632B8B47" Ref="R11"  Part="1"
+AR Path="/63FE6097/632B8B47" Ref="R74"  Part="1"
+F 0 "R10" H 4675 3725 50  0000 C CNN
+F 1 "120" H 4675 3650 50  0000 C CNN
+F 2 "Resistor_SMD:R_0603_1608Metric" H 4800 3700 50  0001 C CNN
+F 3 "~" H 4800 3700 50  0001 C CNN
+	1    4800 3700
+	1    0    0    -1
+$EndComp
+Text HLabel 4675 3475 0    50   Input ~ 0
+LED
+Wire Wire Line
+	4675 3475 4800 3475
+Wire Wire Line
+	4800 3475 4800 3600
 $EndSCHEMATC

Commit message: fixed net names
Parts:
- D14: value OUT 1 -> Servo
- J9: value Servo 1 -> Servo
Changed lines of the file:
@@
 $Descr A4 11693 8268
 encoding utf-8
-Sheet 4 18
+Sheet 14 18
 Title ""
 Date ""
@@
 AR Path="/63F9E75F/63587B1C" Ref="J18"  Part="1"
 AR Path="/63FE6097/63587B1C" Ref="J19"  Part="1"
-F 0 "J9" H 6300 3625 50  0000 C CNN
-F 1 "Servo 1" H 6300 3550 50  0000 C CNN
+F 0 "J19" H 6300 3625 50  0000 C CNN
+F 1 "Servo" H 6300 3550 50  0000 C CNN
 F 2 "TXV_LIB:Molex_Nano-Fit_105309-xx04_1x04_P2.50mm_Vertical" H 6300 3350 50  0001 C CNN
 F 3 "~" H 6300 3350 50  0001 C CNN
@@
 AR Path="/63F9E75F/63587B22" Ref="#PWR0166"  Part="1"
 AR Path="/63FE6097/63587B22" Ref="#PWR0171"  Part="1"
-F 0 "#PWR0114" H 6300 3575 50  0001 C CNN
+F 0 "#PWR0171" H 6300 3575 50  0001 C CNN
 F 1 "GND" H 6300 3675 50  0000 C CNN
 F 2 "" H 6300 3825 50  0001 C CNN
@@
 AR Path="/63F9E75F/63587B2C" Ref="#PWR0167"  Part="1"
 AR Path="/63FE6097/63587B2C" Ref="#PWR0172"  Part="1"
-F 0 "#PWR0115" H 5225 3525 50  0001 C CNN
+F 0 "#PWR0172" H 5225 3525 50  0001 C CNN
 F 1 "GND" H 5225 3625 50  0000 C CNN
 F 2 "" H 5225 3775 50  0001 C CNN
@@
 AR Path="/63F9E75F/63587B33" Ref="R51"  Part="1"
 AR Path="/63FE6097/63587B33" Ref="R54"  Part="1"
-F 0 "R25" H 5166 3354 50  0000 R CNN
+F 0 "R54" H 5166 3354 50  0000 R CNN
 F 1 "9k1" H 5166 3445 50  0000 R CNN
 F 2 "Resistor_SMD:R_0603_1608Metric" H 5225 3400 50  0001 C CNN
@@
 AR Path="/63F9E75F/63587B41" Ref="R52"  Part="1"
 AR Path="/63FE6097/63587B41" Ref="R55"  Part="1"
-F 0 "R26" V 5750 3575 50  0000 L CNN
+F 0 "R55" V 5750 3575 50  0000 L CNN
 F 1 "10m 1W" V 5900 3475 50  0000 L CNN
 F 2 "Resistor_SMD:R_1206_3216Metric" H 5825 3650 50  0001 C CNN
@@
 AR Path="/63F9E75F/63587B47" Ref="R53"  Part="1"
 AR Path="/63FE6097/63587B47" Ref="R56"  Part="1"
-F 0 "R27" V 6000 3575 50  0000 R CNN
+F 0 "R56" V 6000 3575 50  0000 R CNN
 F 1 "1k" V 6025 3425 50  0000 R CNN
 F 2 "Resistor_SMD:R_0603_1608Metric" H 5950 3350 50  0001 C CNN
@@
 AR Path="/63F9E75F/63587B4F" Ref="C56"  Part="1"
 AR Path="/63FE6097/63587B4F" Ref="C58"  Part="1"
-F 0 "C43" H 5025 3675 50  0000 L CNN
+F 0 "C58" H 5025 3675 50  0000 L CNN
 F 1 "100n" H 5025 3575 50  0000 L CNN
 F 2 "Capacitor_SMD:C_0402_1005Metric" H 5225 3650 50  0001 C CNN
@@
 AR Path="/63F9E75F/63587B59" Ref="U16"  Part="1"
 AR Path="/63FE6097/63587B59" Ref="U17"  Part="1"
-F 0 "U10" V 5825 3750 50  0000 L CNN
+F 0 "U17" V 5825 3750 50  0000 L CNN
 F 1 "INA180B1" V 5925 3575 50  0000 L CNN
 F 2 "Package_TO_SOT_SMD:SOT-23-5" H 5875 4075 50  0001 C CNN
@@
 AR Path="/63F9E75F/63587B5F" Ref="#PWR0168"  Part="1"
 AR Path="/63FE6097/63587B5F" Ref="#PWR0173"  Part="1"
-F 0 "#PWR0116" H 5425 3750 50  0001 C CNN
+F 0 "#PWR0173" H 5425 3750 50  0001 C CNN
 F 1 "+3V3" H 5425 4050 50  0000 C CNN
 F 2 "" H 5425 3900 50  0001 C CNN
@@
 AR Path="/63F9E75F/63587B66" Ref="C57"  Part="1"
 AR Path="/63FE6097/63587B66" Ref="C59"  Part="1"
-F 0 "C44" H 5425 4125 50  0000 C CNN
+F 0 "C59" H 5425 4125 50  0000 C CNN
 F 1 "100n" H 5375 3975 50  0000 C CNN
 F 2 "Capacitor_SMD:C_0402_1005Metric" H 5500 4050 50  0001 C CNN
@@
 AR Path="/63F9E75F/63587B6D" Ref="#PWR0169"  Part="1"
 AR Path="/63FE6097/63587B6D" Ref="#PWR0174"  Part="1"
-F 0 "#PWR0117" H 5500 3925 50  0001 C CNN
+F 0 "#PWR0174" H 5500 3925 50  0001 C CNN
 F 1 "GND" H 5500 4025 50  0000 C CNN
 F 2 "" H 5500 4175 50  0001 C CNN
@@
 AR Path="/63F9E75F/62FB5B89" Ref="#PWR0170"  Part="1"
 AR Path="/63FE6097/62FB5B89" Ref="#PWR0175"  Part="1"
-F 0 "#PWR0118" H 5450 3500 50  0001 C CNN
+F 0 "#PWR0175" H 5450 3500 50  0001 C CNN
 F 1 "VS" V 5650 3775 50  0000 L CNN
 F 2 "" H 5650 3650 50  0001 C CNN
@@
 AR Path="/63F9E75F/632B8B39" Ref="D15"  Part="1"
 AR Path="/63FE6097/632B8B39" Ref="D16"  Part="1"
-F 0 "D14" V 4825 4125 50  0000 R CNN
-F 1 "OUT 1" V 4750 4225 50  0000 R CNN
+F 0 "D16" V 4825 4125 50  0000 R CNN
+F 1 "Servo" V 4750 4175 50  0000 R CNN
 F 2 "LED_SMD:LED_0603_1608Metric" V 4800 3925 50  0001 C CNN
 F 3 "~" V 4800 3925 50  0001 C CNN
@@
 AR Path="/63F9E75F/632B8B3F" Ref="#PWR0210"  Part="1"
 AR Path="/63FE6097/632B8B3F" Ref="#PWR0211"  Part="1"
-F 0 "#PWR0209" H 4800 3800 50  0001 C CNN
+F 0 "#PWR0211" H 4800 3800 50  0001 C CNN
 F 1 "GND" H 4800 3900 50  0000 C CNN
 F 2 "" H 4800 4050 50  0001 C CNN
@@
 AR Path="/63F9E75F/632B8B47" Ref="R11"  Part="1"
 AR Path="/63FE6097/632B8B47" Ref="R74"  Part="1"
-F 0 "R10" H 4675 3725 50  0000 C CNN
+F 0 "R74" H 4675 3725 50  0000 C CNN
 F 1 "120" H 4675 3650 50  0000 C CNN
 F 2 "Resistor_SMD:R_0603_1608Metric" H 4800 3700 50  0001 C CNN

Commit message: schematic done, preliminary placement done
Changed lines of the file:
@@
 AR Path="/63F9E75F/63587B1C" Ref="J18"  Part="1"
 AR Path="/63FE6097/63587B1C" Ref="J19"  Part="1"
-F 0 "J19" H 6300 3625 50  0000 C CNN
+F 0 "J18" H 6300 3625 50  0000 C CNN
 F 1 "Servo" H 6300 3550 50  0000 C CNN
 F 2 "TXV_LIB:Molex_Nano-Fit_105309-xx04_1x04_P2.50mm_Vertical" H 6300 3350 50  0001 C CNN
@@
 AR Path="/63F9E75F/63587B22" Ref="#PWR0166"  Part="1"
 AR Path="/63FE6097/63587B22" Ref="#PWR0171"  Part="1"
-F 0 "#PWR0171" H 6300 3575 50  0001 C CNN
+F 0 "#PWR0166" H 6300 3575 50  0001 C CNN
 F 1 "GND" H 6300 3675 50  0000 C CNN
 F 2 "" H 6300 3825 50  0001 C CNN
@@
 AR Path="/63F9E75F/63587B2C" Ref="#PWR0167"  Part="1"
 AR Path="/63FE6097/63587B2C" Ref="#PWR0172"  Part="1"
-F 0 "#PWR0172" H 5225 3525 50  0001 C CNN
+F 0 "#PWR0167" H 5225 3525 50  0001 C CNN
 F 1 "GND" H 5225 3625 50  0000 C CNN
 F 2 "" H 5225 3775 50  0001 C CNN
@@
 AR Path="/63F9E75F/63587B33" Ref="R51"  Part="1"
 AR Path="/63FE6097/63587B33" Ref="R54"  Part="1"
-F 0 "R54" H 5166 3354 50  0000 R CNN
+F 0 "R51" H 5166 3354 50  0000 R CNN
 F 1 "9k1" H 5166 3445 50  0000 R CNN
 F 2 "Resistor_SMD:R_0603_1608Metric" H 5225 3400 50  0001 C CNN
@@
 AR Path="/63F9E75F/63587B41" Ref="R52"  Part="1"
 AR Path="/63FE6097/63587B41" Ref="R55"  Part="1"
-F 0 "R55" V 5750 3575 50  0000 L CNN
+F 0 "R52" V 5750 3575 50  0000 L CNN
 F 1 "10m 1W" V 5900 3475 50  0000 L CNN
 F 2 "Resistor_SMD:R_1206_3216Metric" H 5825 3650 50  0001 C CNN
@@
 AR Path="/63F9E75F/63587B47" Ref="R53"  Part="1"
 AR Path="/63FE6097/63587B47" Ref="R56"  Part="1"
-F 0 "R56" V 6000 3575 50  0000 R CNN
+F 0 "R53" V 6000 3575 50  0000 R CNN
 F 1 "1k" V 6025 3425 50  0000 R CNN
 F 2 "Resistor_SMD:R_0603_1608Metric" H 5950 3350 50  0001 C CNN
@@
 AR Path="/63F9E75F/63587B4F" Ref="C56"  Part="1"
 AR Path="/63FE6097/63587B4F" Ref="C58"  Part="1"
-F 0 "C58" H 5025 3675 50  0000 L CNN
+F 0 "C56" H 5025 3675 50  0000 L CNN
 F 1 "100n" H 5025 3575 50  0000 L CNN
 F 2 "Capacitor_SMD:C_0402_1005Metric" H 5225 3650 50  0001 C CNN
@@
 AR Path="/63F9E75F/63587B59" Ref="U16"  Part="1"
 AR Path="/63FE6097/63587B59" Ref="U17"  Part="1"
-F 0 "U17" V 5825 3750 50  0000 L CNN
+F 0 "U16" V 5825 3750 50  0000 L CNN
 F 1 "INA180B1" V 5925 3575 50  0000 L CNN
 F 2 "Package_TO_SOT_SMD:SOT-23-5" H 5875 4075 50  0001 C CNN
@@
 AR Path="/63F9E75F/63587B5F" Ref="#PWR0168"  Part="1"
 AR Path="/63FE6097/63587B5F" Ref="#PWR0173"  Part="1"
-F 0 "#PWR0173" H 5425 3750 50  0001 C CNN
+F 0 "#PWR0168" H 5425 3750 50  0001 C CNN
 F 1 "+3V3" H 5425 4050 50  0000 C CNN
 F 2 "" H 5425 3900 50  0001 C CNN
@@
 AR Path="/63F9E75F/63587B66" Ref="C57"  Part="1"
 AR Path="/63FE6097/63587B66" Ref="C59"  Part="1"
-F 0 "C59" H 5425 4125 50  0000 C CNN
+F 0 "C57" H 5425 4125 50  0000 C CNN
 F 1 "100n" H 5375 3975 50  0000 C CNN
 F 2 "Capacitor_SMD:C_0402_1005Metric" H 5500 4050 50  0001 C CNN
@@
 AR Path="/63F9E75F/63587B6D" Ref="#PWR0169"  Part="1"
 AR Path="/63FE6097/63587B6D" Ref="#PWR0174"  Part="1"
-F 0 "#PWR0174" H 5500 3925 50  0001 C CNN
+F 0 "#PWR0169" H 5500 3925 50  0001 C CNN
 F 1 "GND" H 5500 4025 50  0000 C CNN
 F 2 "" H 5500 4175 50  0001 C CNN
@@
 AR Path="/63F9E75F/62FB5B89" Ref="#PWR0170"  Part="1"
 AR Path="/63FE6097/62FB5B89" Ref="#PWR0175"  Part="1"
-F 0 "#PWR0175" H 5450 3500 50  0001 C CNN
+F 0 "#PWR0170" H 5450 3500 50  0001 C CNN
 F 1 "VS" V 5650 3775 50  0000 L CNN
 F 2 "" H 5650 3650 50  0001 C CNN
@@
 AR Path="/63F9E75F/632B8B39" Ref="D15"  Part="1"
 AR Path="/63FE6097/632B8B39" Ref="D16"  Part="1"
-F 0 "D16" V 4825 4125 50  0000 R CNN
+F 0 "D15" V 4825 4125 50  0000 R CNN
 F 1 "Servo" V 4750 4175 50  0000 R CNN
 F 2 "LED_SMD:LED_0603_1608Metric" V 4800 3925 50  0001 C CNN
@@
 AR Path="/63F9E75F/632B8B3F" Ref="#PWR0210"  Part="1"
 AR Path="/63FE6097/632B8B3F" Ref="#PWR0211"  Part="1"
-F 0 "#PWR0211" H 4800 3800 50  0001 C CNN
+F 0 "#PWR0210" H 4800 3800 50  0001 C CNN
 F 1 "GND" H 4800 3900 50  0000 C CNN
 F 2 "" H 4800 4050 50  0001 C CNN
@@
 AR Path="/63F9E75F/632B8B47" Ref="R11"  Part="1"
 AR Path="/63FE6097/632B8B47" Ref="R74"  Part="1"
-F 0 "R74" H 4675 3725 50  0000 C CNN
+F 0 "R11" H 4675 3725 50  0000 C CNN
 F 1 "120" H 4675 3650 50  0000 C CNN
 F 2 "Resistor_SMD:R_0603_1608Metric" H 4800 3700 50  0001 C CNN

Commit message: routing done, drc clean (3 errors to be ignored)
Changed lines of the file:
@@
 $Descr A4 11693 8268
 encoding utf-8
-Sheet 18 18
+Sheet 17 18
 Title ""
 Date ""
@@
 AR Path="/63F9E75F/63587B1C" Ref="J18"  Part="1"
 AR Path="/63FE6097/63587B1C" Ref="J19"  Part="1"
-F 0 "J18" H 6300 3625 50  0000 C CNN
+F 0 "J19" H 6300 3625 50  0000 C CNN
 F 1 "Servo" H 6300 3550 50  0000 C CNN
 F 2 "TXV_LIB:Molex_Nano-Fit_105309-xx04_1x04_P2.50mm_Vertical" H 6300 3350 50  0001 C CNN
@@
 AR Path="/63F9E75F/63587B22" Ref="#PWR0166"  Part="1"
 AR Path="/63FE6097/63587B22" Ref="#PWR0171"  Part="1"
-F 0 "#PWR0166" H 6300 3575 50  0001 C CNN
+F 0 "#PWR0171" H 6300 3575 50  0001 C CNN
 F 1 "GND" H 6300 3675 50  0000 C CNN
 F 2 "" H 6300 3825 50  0001 C CNN
@@
 AR Path="/63F9E75F/63587B2C" Ref="#PWR0167"  Part="1"
 AR Path="/63FE6097/63587B2C" Ref="#PWR0172"  Part="1"
-F 0 "#PWR0167" H 5225 3525 50  0001 C CNN
+F 0 "#PWR0172" H 5225 3525 50  0001 C CNN
 F 1 "GND" H 5225 3625 50  0000 C CNN
 F 2 "" H 5225 3775 50  0001 C CNN
@@
 AR Path="/63F9E75F/63587B33" Ref="R51"  Part="1"
 AR Path="/63FE6097/63587B33" Ref="R54"  Part="1"
-F 0 "R51" H 5166 3354 50  0000 R CNN
+F 0 "R54" H 5166 3354 50  0000 R CNN
 F 1 "9k1" H 5166 3445 50  0000 R CNN
 F 2 "Resistor_SMD:R_0603_1608Metric" H 5225 3400 50  0001 C CNN
@@
 AR Path="/63F9E75F/63587B41" Ref="R52"  Part="1"
 AR Path="/63FE6097/63587B41" Ref="R55"  Part="1"
-F 0 "R52" V 5750 3575 50  0000 L CNN
+F 0 "R55" V 5750 3575 50  0000 L CNN
 F 1 "10m 1W" V 5900 3475 50  0000 L CNN
 F 2 "Resistor_SMD:R_1206_3216Metric" H 5825 3650 50  0001 C CNN
@@
 AR Path="/63F9E75F/63587B47" Ref="R53"  Part="1"
 AR Path="/63FE6097/63587B47" Ref="R56"  Part="1"
-F 0 "R53" V 6000 3575 50  0000 R CNN
+F 0 "R56" V 6000 3575 50  0000 R CNN
 F 1 "1k" V 6025 3425 50  0000 R CNN
 F 2 "Resistor_SMD:R_0603_1608Metric" H 5950 3350 50  0001 C CNN
@@
 AR Path="/63F9E75F/63587B4F" Ref="C56"  Part="1"
 AR Path="/63FE6097/63587B4F" Ref="C58"  Part="1"
-F 0 "C56" H 5025 3675 50  0000 L CNN
+F 0 "C58" H 5025 3675 50  0000 L CNN
 F 1 "100n" H 5025 3575 50  0000 L CNN
 F 2 "Capacitor_SMD:C_0402_1005Metric" H 5225 3650 50  0001 C CNN
@@
 AR Path="/63F9E75F/63587B59" Ref="U16"  Part="1"
 AR Path="/63FE6097/63587B59" Ref="U17"  Part="1"
-F 0 "U16" V 5825 3750 50  0000 L CNN
+F 0 "U17" V 5825 3750 50  0000 L CNN
 F 1 "INA180B1" V 5925 3575 50  0000 L CNN
 F 2 "Package_TO_SOT_SMD:SOT-23-5" H 5875 4075 50  0001 C CNN
@@
 AR Path="/63F9E75F/63587B5F" Ref="#PWR0168"  Part="1"
 AR Path="/63FE6097/63587B5F" Ref="#PWR0173"  Part="1"
-F 0 "#PWR0168" H 5425 3750 50  0001 C CNN
+F 0 "#PWR0173" H 5425 3750 50  0001 C CNN
 F 1 "+3V3" H 5425 4050 50  0000 C CNN
 F 2 "" H 5425 3900 50  0001 C CNN
@@
 AR Path="/63F9E75F/63587B66" Ref="C57"  Part="1"
 AR Path="/63FE6097/63587B66" Ref="C59"  Part="1"
-F 0 "C57" H 5425 4125 50  0000 C CNN
+F 0 "C59" H 5425 4125 50  0000 C CNN
 F 1 "100n" H 5375 3975 50  0000 C CNN
 F 2 "Capacitor_SMD:C_0402_1005Metric" H 5500 4050 50  0001 C CNN
@@
 AR Path="/63F9E75F/63587B6D" Ref="#PWR0169"  Part="1"
 AR Path="/63FE6097/63587B6D" Ref="#PWR0174"  Part="1"
-F 0 "#PWR0169" H 5500 3925 50  0001 C CNN
+F 0 "#PWR0174" H 5500 3925 50  0001 C CNN
 F 1 "GND" H 5500 4025 50  0000 C CNN
 F 2 "" H 5500 4175 50  0001 C CNN
@@
 AR Path="/63F9E75F/62FB5B89" Ref="#PWR0170"  Part="1"
 AR Path="/63FE6097/62FB5B89" Ref="#PWR0175"  Part="1"
-F 0 "#PWR0170" H 5450 3500 50  0001 C CNN
+F 0 "#PWR0175" H 5450 3500 50  0001 C CNN
 F 1 "VS" V 5650 3775 50  0000 L CNN
 F 2 "" H 5650 3650 50  0001 C CNN
@@
 AR Path="/63F9E75F/632B8B39" Ref="D15"  Part="1"
 AR Path="/63FE6097/632B8B39" Ref="D16"  Part="1"
-F 0 "D15" V 4825 4125 50  0000 R CNN
+F 0 "D16" V 4825 4125 50  0000 R CNN
 F 1 "Servo" V 4750 4175 50  0000 R CNN
 F 2 "LED_SMD:LED_0603_1608Metric" V 4800 3925 50  0001 C CNN
@@
 AR Path="/63F9E75F/632B8B3F" Ref="#PWR0210"  Part="1"
 AR Path="/63FE6097/632B8B3F" Ref="#PWR0211"  Part="1"
-F 0 "#PWR0210" H 4800 3800 50  0001 C CNN
+F 0 "#PWR0211" H 4800 3800 50  0001 C CNN
 F 1 "GND" H 4800 3900 50  0000 C CNN
 F 2 "" H 4800 4050 50  0001 C CNN
@@
 AR Path="/63F9E75F/632B8B47" Ref="R11"  Part="1"
 AR Path="/63FE6097/632B8B47" Ref="R74"  Part="1"
-F 0 "R11" H 4675 3725 50  0000 C CNN
+F 0 "R74" H 4675 3725 50  0000 C CNN
 F 1 "120" H 4675 3650 50  0000 C CNN
 F 2 "Resistor_SMD:R_0603_1608Metric" H 4800 3700 50  0001 C CNN
