File: ServoOutput.sch (KiCad schematic (older format))
At the start: 9 parts, among them J9 Servo, U10 INA180B1

Commit message: some more small changes
Parts:
- R25: value 9k1 -> 10k
Changed lines of the file:
@@
 $Descr A4 11693 8268
 encoding utf-8
-Sheet 17 18
+Sheet 18 18
 Title ""
 Date ""
@@
 AR Path="/63FE6097/63587B33" Ref="R54"  Part="1"
 F 0 "R51" H 5166 3354 50  0000 R CNN
-F 1 "9k1" H 5166 3445 50  0000 R CNN
+F 1 "10k" H 5166 3445 50  0000 R CNN
 F 2 "Resistor_SMD:R_0603_1608Metric" H 5225 3400 50  0001 C CNN
 F 3 "~" H 5225 3400 50  0001 C CNN
