File: PyroOutput.sch (KiCad schematic (older format))
At the start: 9 parts, among them J11 Pyro, U11 TPS1HC100

Commit message: small changes, generated gerbers
Parts:
- R34: value 22k -> 56k
- R36: value 100k -> 56k
Changed lines of the file:
@@
 $Descr A4 11693 8268
 encoding utf-8
-Sheet 14 18
+Sheet 6 18
 Title ""
 Date ""
@@
 AR Path="/64156100/639C464D" Ref="R64"  Part="1"
 AR Path="/6419F64A/639C464D" Ref="R69"  Part="1"
-F 0 "R69" H 6250 4425 50  0000 R CNN
+F 0 "R35" H 6250 4425 50  0000 R CNN
 F 1 "1k" H 6250 4500 50  0000 R CNN
 F 2 "Resistor_SMD:R_0603_1608Metric" H 6300 4450 50  0001 C CNN
@@
 AR Path="/64156100/639C4656" Ref="#PWR0180"  Part="1"
 AR Path="/6419F64A/639C4656" Ref="#PWR0187"  Part="1"
-F 0 "#PWR0187" H 4875 3625 50  0001 C CNN
+F 0 "#PWR0123" H 4875 3625 50  0001 C CNN
 F 1 "GND" V 4875 3675 50  0000 C CNN
 F 2 "" H 4875 3875 50  0001 C CNN
@@
 AR Path="/64156100/639C465D" Ref="#PWR0181"  Part="1"
 AR Path="/6419F64A/639C465D" Ref="#PWR0188"  Part="1"
-F 0 "#PWR0188" H 5150 3550 50  0001 C CNN
+F 0 "#PWR0124" H 5150 3550 50  0001 C CNN
 F 1 "Pyro" H 5150 3850 50  0000 C CNN
 F 2 "" H 5150 3700 50  0001 C CNN
@@
 AR Path="/64156100/639C4663" Ref="C60"  Part="1"
 AR Path="/6419F64A/639C4663" Ref="C61"  Part="1"
-F 0 "C61" V 4900 3825 50  0000 L CNN
+F 0 "C45" V 4900 3825 50  0000 L CNN
 F 1 "100n" V 5100 3775 50  0000 L CNN
 F 2 "Capacitor_SMD:C_0402_1005Metric" H 5000 3875 50  0001 C CNN
@@
 AR Path="/64156100/639C466C" Ref="#PWR0182"  Part="1"
 AR Path="/6419F64A/639C466C" Ref="#PWR0189"  Part="1"
-F 0 "#PWR0189" H 5200 4025 50  0001 C CNN
+F 0 "#PWR0125" H 5200 4025 50  0001 C CNN
 F 1 "+3V3" V 5200 4400 50  0000 C CNN
 F 2 "" H 5200 4175 50  0001 C CNN
@@
 AR Path="/64156100/639C4675" Ref="R62"  Part="1"
 AR Path="/6419F64A/639C4675" Ref="R67"  Part="1"
-F 0 "R67" H 5050 4400 50  0000 R CNN
+F 0 "R33" H 5050 4400 50  0000 R CNN
 F 1 "56k" H 5050 4475 50  0000 R CNN
 F 2 "Resistor_SMD:R_0603_1608Metric" H 5100 4425 50  0001 C CNN
@@
 AR Path="/64156100/639C468D" Ref="#PWR0183"  Part="1"
 AR Path="/6419F64A/639C468D" Ref="#PWR0190"  Part="1"
-F 0 "#PWR0190" H 6300 4325 50  0001 C CNN
+F 0 "#PWR0126" H 6300 4325 50  0001 C CNN
 F 1 "GND" H 6300 4425 50  0000 C CNN
 F 2 "" H 6300 4575 50  0001 C CNN
@@
 AR Path="/64156100/639C469C" Ref="U18"  Part="1"
 AR Path="/6419F64A/639C469C" Ref="U19"  Part="1"
-F 0 "U19" H 5675 4900 50  0000 C CNN
+F 0 "U11" H 5675 4900 50  0000 C CNN
 F 1 "TPS1HC100" H 5675 4825 50  0000 C CNN
 F 2 "Package_SO:HTSSOP-14-1EP_4.4x5mm_P0.65mm_EP3.4x5mm_Mask3x3.1mm" H 5675 3575 50  0001 C CNN
@@
 AR Path="/64156100/639C46A2" Ref="R61"  Part="1"
 AR Path="/6419F64A/639C46A2" Ref="R66"  Part="1"
-F 0 "R66" H 4700 4225 50  0000 C CNN
+F 0 "R32" H 4700 4225 50  0000 C CNN
 F 1 "120" H 4700 4150 50  0000 C CNN
 F 2 "Resistor_SMD:R_0603_1608Metric" H 4825 4200 50  0001 C CNN
@@
 AR Path="/64156100/639C46AD" Ref="R65"  Part="1"
 AR Path="/6419F64A/639C46AD" Ref="R70"  Part="1"
-F 0 "R70" V 6600 3575 50  0000 L CNN
-F 1 "100k" V 6525 3575 50  0000 L CNN
+F 0 "R36" V 6600 3575 50  0000 L CNN
+F 1 "56k" V 6525 3575 50  0000 L CNN
 F 2 "Resistor_SMD:R_0603_1608Metric" H 6450 3650 50  0001 C CNN
 F 3 "~" H 6450 3650 50  0001 C CNN
@@
 AR Path="/64156100/639C46B3" Ref="R63"  Part="1"
 AR Path="/6419F64A/639C46B3" Ref="R68"  Part="1"
-F 0 "R68" V 6050 3650 50  0000 C CNN
-F 1 "22k" V 6125 3650 50  0000 C CNN
+F 0 "R34" V 6050 3650 50  0000 C CNN
+F 1 "56k" V 6125 3650 50  0000 C CNN
 F 2 "Resistor_SMD:R_0603_1608Metric" H 6200 3650 50  0001 C CNN
 F 3 "~" H 6200 3650 50  0001 C CNN
@@
 AR Path="/64156100/639C46B9" Ref="#PWR0184"  Part="1"
 AR Path="/6419F64A/639C46B9" Ref="#PWR0191"  Part="1"
-F 0 "#PWR0191" H 6075 3400 50  0001 C CNN
+F 0 "#PWR0127" H 6075 3400 50  0001 C CNN
 F 1 "+3V3" H 6075 3700 50  0000 C CNN
 F 2 "" H 6075 3550 50  0001 C CNN
@@
 AR Path="/64156100/639C46CD" Ref="#PWR0185"  Part="1"
 AR Path="/6419F64A/639C46CD" Ref="#PWR0192"  Part="1"
-F 0 "#PWR0192" H 6300 3775 50  0001 C CNN
+F 0 "#PWR0128" H 6300 3775 50  0001 C CNN
 F 1 "GND" H 6300 3875 50  0000 C CNN
 F 2 "" H 6300 4025 50  0001 C CNN
@@
 AR Path="/64156100/639C46D4" Ref="#PWR0186"  Part="1"
 AR Path="/6419F64A/639C46D4" Ref="#PWR0193"  Part="1"
-F 0 "#PWR0193" H 5150 4500 50  0001 C CNN
+F 0 "#PWR0129" H 5150 4500 50  0001 C CNN
 F 1 "GND" H 5150 4600 50  0000 C CNN
 F 2 "" H 5150 4750 50  0001 C CNN
@@
 AR Path="/64156100/639C46DA" Ref="D11"  Part="1"
 AR Path="/6419F64A/639C46DA" Ref="D12"  Part="1"
-F 0 "D12" V 4850 4675 50  0000 R CNN
+F 0 "D8" V 4850 4675 50  0000 R CNN
 F 1 "PYRO 1" V 4775 4775 50  0000 R CNN
 F 2 "LED_SMD:LED_0603_1608Metric" V 4825 4425 50  0001 C CNN
@@
 AR Path="/64156100/639C46E3" Ref="J21"  Part="1"
 AR Path="/6419F64A/639C46E3" Ref="J22"  Part="1"
-F 0 "J22" H 6630 3967 50  0000 L CNN
+F 0 "J11" H 6630 3967 50  0000 L CNN
 F 1 "Pyro" H 6630 3876 50  0000 L CNN
 F 2 "TXV_LIB:Molex_SL_1x2_Vertical" H 6550 3975 50  0001 C CNN
