File: TemperatureSensorInput.sch (KiCad schematic (older format))
At the start: 4 parts, among them J8 TEMP

Commit message: some more small changes
Parts:
- R71: value 9k1 -> 10k
Changed lines of the file:
@@
 $Descr A4 11693 8268
 encoding utf-8
-Sheet 11 18
+Sheet 12 18
 Title ""
 Date ""
@@
 AR Path="/63E36C88/61BD0A9D" Ref="R73"  Part="1"
 F 0 "R73" V 6150 3675 50  0000 L CNN
-F 1 "9k1" V 6150 3850 50  0000 L CNN
+F 1 "10k" V 6150 3850 50  0000 L CNN
 F 2 "Resistor_SMD:R_0603_1608Metric" H 6075 3825 50  0001 C CNN
 F 3 "~" H 6075 3825 50  0001 C CNN
