File: uHoubolt_PCB_ECU.kicad_pcb (KiCad board)
At the start: 4 copper layers, 70 x 40 mm, 212 parts, among them J1 Power In, J10 OUT 1, J11 PYRO 1, J12 Pressure 1, J13 Pressure 1, J14 Pressure 1, J15 Pressure 1, J16 TEMP 1, J17 TEMP 1, J18 Servo 1, J19 Servo 1, J2 Debug, J20 OUT 1, J21 PYRO 1, J22 PYRO 1, J23 Pressure 1, J24 12V, J25 GND, J26 Servo, J3 CAN1, J35 CAN1, J36 CAN2, J37 CAN1, J38 CAN2, J4 CAN2, J5 CAN1, J6 CAN2, J7 Pressure 1, J8 TEMP 1, J9 Servo 1, Q1 SISA88DN or similar, Q2 SISA88DN or similar, U1 INA180B1, U10 INA180B1, U11 TPS1HC100, U12 INA180B1, U13 INA180B1, U14 INA180B1, U15 INA180B1, U16 INA180B1, U17 INA180B1, U18 TPS1HC100, U19 TPS1HC100, U2 TS30041-M050QFNR, U20 D1213A-04V, U3 MCP1700-3302E, U4 MCP2562FDT-H_SN, U5 MCP2562FDT, U6 STM32G491MET6-LQFP80, U7 ICM-20602, U8 W25Q256JV, U9 INA180B1, X1 TXC-7C

Commit message: fixed net names
Parts:
- D14, D15, D16: value OUT 1 -> Servo
- J10, J20: value OUT 1 -> Solenoid
- J11, J21, J22: value PYRO 1 -> Pyro
- J12, J13, J14, J15, J23, J7: value Pressure 1 -> Pressure
- J16, J17, J8: value TEMP 1 -> TEMP
- J18, J19, J9: value Servo 1 -> Servo
Connections:
- net /OUT_2_CTRL renamed /OUT_0_CTRL
- net /TEMP_3 renamed /TEMP_0
- net /UART4_RX renamed /UART_RX
- net /UART4_TX renamed /UART_TX
- C2 pad 1: /PRESS_6 -> /PRESS_2
- C41 pad 1: /PRESS_1 -> /PRESS_0
- C43 pad 1: /SERVO_1_FDBK -> /SERVO_0_FDBK
- C47 pad 1: /PRESS_2 -> /PRESS_5
- C49 pad 1: /PRESS_3 -> /PRESS_4
- C51 pad 1: /PRESS_4 -> /PRESS_3
- C53 pad 1: /PRESS_5 -> /PRESS_1
- C58 pad 1: /SERVO_3_FDBK -> /SERVO_1_FDBK
- Q1 pad 3: /OUT_2_CURR -> /OUT_1_CURR
- Q2 pad 3: /OUT_2_CURR -> /OUT_0_CURR
- R10 pad 1: /SERVO_1_LED -> /SERVO_0_LED
- R23 pad 2: /PRESS_1 -> /PRESS_0
- R25 pad 1: /SERVO_1_FDBK -> /SERVO_0_FDBK
- R27 pad 1: /SERVO_1_PWM -> /SERVO_0_PWM
- R31 pad 1: /OUT_2_CURR -> /OUT_1_CURR
- R32 pad 1: /PYRO_1_CTRL -> /PYRO_0_CTRL
- R35 pad 2: /PYRO_1_CURR -> /PYRO_0_CURR
- R36 pad 1: /PYRO_1_CONT -> /PYRO_0_CONT
- R39 pad 2: /PRESS_2 -> /PRESS_5
- R42 pad 2: /PRESS_3 -> /PRESS_4
- R45 pad 2: /PRESS_4 -> /PRESS_3
- R48 pad 2: /PRESS_5 -> /PRESS_1
- R54 pad 1: /SERVO_3_FDBK -> /SERVO_1_FDBK
- R56 pad 1: /SERVO_3_PWM -> /SERVO_1_PWM
- R60 pad 1: /OUT_2_CURR -> /OUT_0_CURR
- R61 pad 1: /PYRO_2_CTRL -> /PYRO_1_CTRL
- R64 pad 2: /PYRO_2_CURR -> /PYRO_1_CURR
- R65 pad 1: /PYRO_2_CONT -> /PYRO_1_CONT
- R66 pad 1: /PYRO_3_CTRL -> /PYRO_2_CTRL
- R69 pad 2: /PYRO_3_CURR -> /PYRO_2_CURR
- R7 pad 2: /PRESS_6 -> /PRESS_2
- R70 pad 1: /PYRO_3_CONT -> /PYRO_2_CONT
- R74 pad 1: /SERVO_3_LED -> /SERVO_1_LED
- U10 pad 4: /SERVO_1_CURR -> /SERVO_0_CURR
- U11 pad 2: /PYRO_1_CTRL -> /PYRO_0_CTRL
- U11 pad 6: /PYRO_1_CURR -> /PYRO_0_CURR
- U17 pad 4: /SERVO_3_CURR -> /SERVO_1_CURR
- U18 pad 2: /PYRO_2_CTRL -> /PYRO_1_CTRL
- U18 pad 6: /PYRO_2_CURR -> /PYRO_1_CURR
- U19 pad 2: /PYRO_3_CTRL -> /PYRO_2_CTRL
- U19 pad 6: /PYRO_3_CURR -> /PYRO_2_CURR

Commit message: schematic done, preliminary placement done
Parts:
- added Q3: SISA88DN or similar, TXV_LIB:PowerPAK_1212-8, F.Cu at (148.9, 107.2)
- added R77: 120, Resistor_SMD:R_0603_1608Metric, F.Cu at (149.9, 103.8)
- added R78: 1k, Resistor_SMD:R_0603_1608Metric, F.Cu at (148.0, 101.4)
- added U21: D1213A-04V, Package_TO_SOT_SMD:SOT-563, F.Cu at (166.1, 88.5)
- added U22: D1213A-04V, Package_TO_SOT_SMD:SOT-563, F.Cu at (170.2, 95.4)
- added U23: D1213A-04V, Package_TO_SOT_SMD:SOT-563, F.Cu at (162.1, 108.5)
- added U24: D1213A-04V, Package_TO_SOT_SMD:SOT-563, F.Cu at (154.9, 108.5)
- moved U20 56.3 mm to (150.6, 90.1), turned to 90 degrees
- moved C55 31.2 mm to (175.2, 97.8)
- moved R50 31.2 mm to (175.2, 96.3)
- moved R73 31.2 mm to (175.2, 94.8)
- moved C42 28.0 mm to (175.2, 102.2)
- moved R24 28.0 mm to (175.2, 100.8)
- moved R71 28.0 mm to (175.2, 99.3)
- moved R49 26.9 mm to (175.2, 105.2)
- moved R72 26.9 mm to (175.2, 103.7)
- moved C54 26.9 mm to (175.2, 106.6)
- moved R19 7.62 mm to (171.1, 106.5)
- moved R20 7.27 mm to (171.1, 108.0)
- moved D4 2.10 mm to (178.1, 103.0)
- moved D5 2.10 mm to (178.1, 105.2)
- moved U7 1.65 mm to (171.6, 102.3)
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Connections:
- LS1 pad 1: /Speaker_P -> +12VA
- LS1 pad 2: /Speaker_N -> Net-(LS1-Pad2)
- Q1 pad 3: /OUT_1_CURR -> /SOLENOID_1_CURR
- Q2 pad 3: /OUT_0_CURR -> /SOLENOID_0_CURR
- R28 pad 1: /OUT_1_CTRL -> /SOLENOID_1_CTRL
- R29 pad 2: /OUT_1_CTRL -> /SOLENOID_1_CTRL
- R30 pad 1: /OUT_1_CTRL -> /SOLENOID_1_CTRL
- R31 pad 1: /OUT_1_CURR -> /SOLENOID_1_CURR
- R57 pad 1: /OUT_0_CTRL -> /SOLENOID_0_CTRL
- R58 pad 2: /OUT_0_CTRL -> /SOLENOID_0_CTRL
- R59 pad 1: /OUT_0_CTRL -> /SOLENOID_0_CTRL
- R60 pad 1: /OUT_0_CURR -> /SOLENOID_0_CURR
- U20 pad 1: Net-(U20-Pad1) -> /SOLENOID_0_CURR
- U20 pad 3: Net-(U20-Pad3) -> /SOLENOID_1_CURR
- U20 pad 4: Net-(U20-Pad4) -> /SERVO_2_FDBK
- U20 pad 6: Net-(U20-Pad6) -> /SERVO_1_FDBK
- U6 pad 10: Net-(U6-Pad10) -> /TEMP_2
- U6 pad 11: Net-(U6-Pad11) -> /SERVO_0_FDBK
- U6 pad 12: Net-(U6-Pad12) -> /SERVO_0_CURR
- U6 pad 13: Net-(U6-Pad13) -> /SERVO_1_FDBK
- U6 pad 14: Net-(U6-Pad14) -> /SERVO_1_CURR
- U6 pad 17: Net-(U6-Pad17) -> /SERVO_2_FDBK
- U6 pad 18: Net-(U6-Pad18) -> /SERVO_2_CURR
- U6 pad 2: Net-(U6-Pad2) -> /SERVO_0_LED
- U6 pad 20: Net-(U6-Pad20) -> /12V_SENSE
- U6 pad 21: Net-(U6-Pad21) -> /SOLENOID_1_CURR
- U6 pad 22: Net-(U6-Pad22) -> /5V_SENSE
- U6 pad 23: Net-(U6-Pad23) -> /12VA_SENSE
- U6 pad 24: Net-(U6-Pad24) -> /SOLENOID_0_CURR
- U6 pad 25: Net-(U6-Pad25) -> /PYRO_SENSE
- U6 pad 3: Net-(U6-Pad3) -> /SERVO_1_LED
- U6 pad 30: Net-(U6-Pad30) -> /PYRO_2_CURR
- U6 pad 31: Net-(U6-Pad31) -> /PYRO_1_CURR
- U6 pad 32: Net-(U6-Pad32) -> /PYRO_0_CURR
- U6 pad 39: Net-(U6-Pad39) -> /Speaker
- U6 pad 4: Net-(U6-Pad4) -> /SERVO_2_LED
- U6 pad 42: Net-(U6-Pad42) -> /PRESS_2
- U6 pad 43: Net-(U6-Pad43) -> /PRESS_5
- U6 pad 44: Net-(U6-Pad44) -> /PRESS_1
- U6 pad 45: Net-(U6-Pad45) -> /PRESS_4
- U6 pad 46: Net-(U6-Pad46) -> /PRESS_0
- U6 pad 47: Net-(U6-Pad47) -> /SOLENOID_0_CTRL
- U6 pad 48: Net-(U6-Pad48) -> /SOLENOID_1_CTRL
- U6 pad 49: Net-(U6-Pad49) -> /PRESS_3
- U6 pad 52: Net-(U6-Pad52) -> /5V_PGOOD
- U6 pad 53: Net-(U6-Pad53) -> /PYRO_2_CTRL
- U6 pad 54: Net-(U6-Pad54) -> /PYRO_2_CONT
- U6 pad 55: Net-(U6-Pad55) -> /PYRO_1_CTRL
- U6 pad 56: Net-(U6-Pad56) -> /PYRO_1_CONT
- U6 pad 57: Net-(U6-Pad57) -> /PYRO_0_CTRL
- U6 pad 58: Net-(U6-Pad58) -> /PYRO_0_CONT
- U6 pad 70: Net-(U6-Pad70) -> /LED_2
- U6 pad 71: Net-(U6-Pad71) -> /LED_1
- U6 pad 72: Net-(U6-Pad72) -> /UART_TX
- U6 pad 73: Net-(U6-Pad73) -> /UART_RX
- U6 pad 76: Net-(U6-Pad76) -> /SERVO_0_PWM
- U6 pad 77: Net-(U6-Pad77) -> /SERVO_1_PWM
- U6 pad 78: Net-(U6-Pad78) -> /SERVO_2_PWM
- U6 pad 8: Net-(U6-Pad8) -> /TEMP_0
- U6 pad 9: Net-(U6-Pad9) -> /TEMP_1
Routing:
- net /5V_PGOOD: track 0.00 -> 0.56 mm, vias 0 -> 1

Commit message: routing started
Parts:
- removed the J1 at (123.5, 100.0)
- J1: footprint TXV_LIB:Molex_MegaFit_1x03_Vertical -> TXV_LIB:Molex_MegaFit_1x03_Vertical_Doublesided
- U20, U21, U22, U23, U24: footprint Package_TO_SOT_SMD:SOT-563 -> TXV_LIB:SOT-563
- moved R69 7.81 mm to (127.9, 109.9), turned to 180 degrees
- moved R67 7.80 mm to (128.3, 117.7), turned to 90 degrees
- moved R20 3.02 mm to (171.4, 105.0), turned to 90 degrees
- moved R19 2.41 mm to (172.9, 105.0), turned to 90 degrees
- moved C36 1.20 mm to (170.8, 97.8)
- moved C37 1.15 mm to (170.9, 99.0)
- moved C40 1.10 mm to (172.8, 98.5)
- moved U7 1.10 mm to (171.7, 101.2)
- moved C39 1.10 mm to (169.4, 99.5)
- moved R77 0.45 mm to (149.5, 103.9)
- moved R36 0.25 mm to (151.9, 109.9)
- moved R32 0.20 mm to (148.9, 109.9)
- moved C54 0.20 mm to (175.2, 106.8)
- moved C38 0.16 mm to (146.7, 104.5)
- moved R35 0.15 mm to (145.9, 109.9)
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Connections:
- LS1 pad 1: +12VA -> +12V
- R78 pad 1: +12VA -> +12V
Routing:
- net +5V: track 0.00 -> 98.3 mm, vias 0 -> 13
- net +12VA: track 0.00 -> 89.5 mm, vias 0 -> 8
- net +3V3: track 17.0 -> 74.1 mm, vias 6 -> 41
- net +12V: track 8.45 -> 39.9 mm, vias 2 -> 7
- net /SWCLK: track 0.00 -> 19.4 mm, vias 0 -> 3
- net /QSPI1_CLK: track 0.00 -> 17.6 mm, vias 0 -> 2
- net /QSPI1_BK1_IO2: track 0.00 -> 16.9 mm, vias 0 -> 2
- net /SWDIO: track 0.00 -> 16.5 mm, vias 0 -> 1
- net /QSPI1_BK1_IO1: track 0.00 -> 16.3 mm, vias 0 -> 2
- net /QSPI1_BK1_NCS: track 0.00 -> 16.0 mm, vias 0 -> 2
- net /SERVO_0_LED: track 0.00 -> 13.2 mm
- net /QSPI1_BK1_IO0: track 0.00 -> 12.9 mm, vias 0 -> 2
- net /UART_TX: track 0.00 -> 12.3 mm, vias 0 -> 1
- net Net-(LS1-Pad2): track 0.00 -> 11.5 mm
- net /QSPI1_BK1_IO3: track 0.00 -> 10.5 mm, vias 0 -> 2
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- added copper zone on In2.Cu, net +12V
- added copper zone on F.Cu, net +12VA
- added copper zone on F.Cu, net +3V3
- added copper zone on F.Cu, net +5V
- added copper zone on F.Cu, net /SOLENOID_0_CURR
- added copper zone on F.Cu, net /SOLENOID_1_CURR
- added copper zone on F.Cu, net Net-(D10-Pad2)
- added copper zone on F.Cu, net Net-(D7-Pad2)
- added copper zone on F.Cu, net Net-(J11-Pad2)
- added copper zone on F.Cu, net Net-(J18-Pad3)
- added copper zone on F.Cu, net Net-(J19-Pad3)
- added copper zone on F.Cu, net Net-(J21-Pad2)
- added copper zone on F.Cu, net Net-(J22-Pad2)
- added copper zone on F.Cu, net Net-(J9-Pad3)
- added copper zone on F.Cu, net Net-(LS1-Pad2)
- added copper zone on F.Cu, net PYRO
- added copper zone on In2.Cu, net PYRO
- added copper zone on B.Cu, net VS
- added copper zone on F.Cu, net VS

Commit message: routing done, drc clean (3 errors to be ignored)
Parts:
- removed J24: 12V, TXV_LIB:PlatedEdgePad_6mm
- removed J25: GND, TXV_LIB:PlatedEdgePad_6mm
- removed J26: Servo, TXV_LIB:PlatedEdgePad_6mm
- added JP2: Servo Voltage Select, TXV_LIB:Jumper3_6x2mm_Vias23, B.Cu at (158.2, 94.3)
- moved U22 1.08 mm to (170.3, 94.3)
- moved C32 0.25 mm to (159.2, 107.8)
- moved C26 0.20 mm to (183.3, 109.5)
- moved R17 0.20 mm to (188.8, 109.6)
- moved U4 0.20 mm to (185.9, 109.6)
- moved C21 0.20 mm to (186.9, 111.8)
- moved R11 0.10 mm to (150.7, 85.8)
- moved X1 0.10 mm to (144.8, 89.9)
Connections:
- U6 pad 21: /SOLENOID_1_CURR -> /SOLENOID_0_CURR
- U6 pad 24: /SOLENOID_0_CURR -> /SOLENOID_1_CURR
- U6 pad 47: /SOLENOID_0_CTRL -> /SOLENOID_1_CTRL
- U6 pad 48: /SOLENOID_1_CTRL -> /SOLENOID_0_CTRL
- U8 pad 9: (no net) -> GND
Routing:
- net /5V_unfused: track 14.4 -> 94.0 mm, vias 2 -> 8
- net /CAN1_H: track 3.22 -> 71.5 mm, vias 0 -> 3
- net /CAN2_L: track 3.22 -> 71.4 mm, vias 0 -> 1
- net /CAN1_L: track 3.22 -> 71.3 mm, vias 0 -> 3
- net /CAN2_H: track 10.1 -> 73.2 mm, vias 0 -> 1
- net +5V: track 98.3 -> 149.1 mm, vias 13 -> 17
- net /PYRO_0_CONT: track 0.00 -> 46.1 mm, vias 0 -> 3
- net /TEMP_2: track 0.00 -> 41.6 mm, vias 0 -> 3
- net /PYRO_SENSE: track 1.35 -> 42.0 mm, vias 0 -> 2
- net /5V_PGOOD: track 0.56 -> 41.0 mm, vias 1 -> 4
- net /SOLENOID_1_CTRL: track 8.43 -> 48.1 mm, vias 2 -> 3
- net /PYRO_1_CTRL: track 5.13 -> 43.8 mm, vias 0 -> 2
- net /SERVO_2_PWM: track 0.00 -> 37.7 mm, vias 0 -> 2
- net /PYRO_2_CTRL: track 4.98 -> 42.4 mm, vias 0 -> 3
- net /PRESS_3: track 1.34 -> 38.4 mm, vias 0 -> 2
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Other:
- board text added: "12V"
- board text added: "GND"
- board text added: "VS"

Commit message: small improvements, updated doc
Parts:
- removed G***: LOGO, TXV_LIB:ST_Logo_new
- added G1: SpaceTeam_LOGO, TXV_LIB:ST_Logo_new, B.Cu at (166.5, 97.2)
Routing:
- net /5V_unfused: track 94.0 -> 91.4 mm
- net /SERVO_1_FDBK: track 35.0 -> 33.7 mm
- net /SERVO_0_LED: track 16.5 -> 15.3 mm
- net +12VA: track 89.6 -> 90.7 mm
- net /SERVO_0_FDBK: track 27.9 -> 26.9 mm
- net /PRESS_1: track 15.8 -> 16.5 mm
- net /SOLENOID_0_CTRL: track 42.8 -> 42.2 mm
- net /PRESS_0: track 25.2 -> 25.8 mm
- net /SERVO_2_CURR: track 14.2 -> 14.8 mm
- net /PYRO_SENSE: track 42.0 -> 41.5 mm
- net GND: track 4.31 -> 4.40 mm, vias 106 -> 111

Commit message: small changes, generated gerbers
Parts:
- R34, R63, R68: value 22k -> 56k
- R36, R65, R70: value 100k -> 56k
- U4: value MCP2562FDT-H_SN -> MCP2562FDx-x_MF
- U5: value MCP2562FDT -> MCP2562FDx-x_MF
- moved D11 0.10 mm to (140.3, 112.3)
- moved D12 0.10 mm to (131.5, 112.3)
- moved D8 0.10 mm to (149.2, 112.3)
Other:
- board text added: "JLCJLCJLCJLC"

Commit message: some more small changes
Parts:
- R1, R21, R37, R40, R43, R46: value 4k7/0 -> 5k6/0
- R12, R4, R8: value 9k1 -> 56k
- R13, R5, R9: value 1k -> 10k
- R14, R15, R16, R23, R25, R29, R39, R42, R45, R48, R51, R54, R58, R7, R71, R72, R73: value 9k1 -> 10k
- R2, R22, R38, R41, R44, R47: value 6k8/160 -> 10k/160
Routing:
- net /TEMP_1: track 28.0 -> 35.7 mm
- net /CAN2_H: track 73.1 -> 68.7 mm
- net /5V_unfused: track 91.4 -> 88.6 mm
- net /CAN2_L: track 71.3 -> 74.1 mm
- net /TEMP_0: track 33.9 -> 31.2 mm
- net +12VA: track 90.7 -> 93.0 mm
- net +5V: track 148.6 -> 150.7 mm
- net /12VA_SENSE: track 28.4 -> 26.6 mm
- net /TEMP_2: track 41.6 -> 39.9 mm
- net /NRST: track 24.9 -> 23.3 mm
- net /SERVO_0_CURR: track 15.4 -> 14.5 mm
- net /PYRO_2_CTRL: track 42.4 -> 43.3 mm
- net Net-(J14-Pad2): track 7.85 -> 8.72 mm
- net GND: track 4.40 -> 4.76 mm, vias 111 -> 147

Commit message: tiny changes, version to be ordered
Other:
- board text added: "Daniel Frank 2021"
