File: PressureSensorInput.kicad_sch (KiCad schematic)
At the start: 8 parts, among them J23 Pressure, U1 INA180B1

Commit message: WIP v1.1, fixed JP2 footprint, replaced STM footprint, re-routing in progress
Parts:
- renumbered C1 to C52, C2 to C53, J23 to J15, JP3 to JP7, R1 to R46, R2 to R47, R7 to R48, U1 to U15
Changed lines of the file:
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@@
   (symbol (lib_id "TXV_LIB:INA180B") (at 144.145 95.885 0)
     (in_bom yes) (on_board yes)
-    (property "Reference" "U1" (id 0) (at 146.685 98.425 0)
+    (property "Reference" "U15" (id 0) (at 146.685 98.425 0)
       (effects (font (size 1.27 1.27)) (justify left))
     )
@@
   (symbol (lib_id "Device:C_Small") (at 145.415 87.63 90)
     (in_bom yes) (on_board yes)
-    (property "Reference" "C1" (id 0) (at 145.415 85.09 90))
+    (property "Reference" "C52" (id 0) (at 145.415 85.09 90))
     (property "Value" "100n" (id 1) (at 145.415 90.805 90))
     (property "Footprint" "Capacitor_SMD:C_0402_1005Metric" (id 2) (at 145.415 87.63 0)
@@
   (symbol (lib_id "Device:R_Small") (at 133.35 101.6 0)
     (in_bom yes) (on_board yes)
-    (property "Reference" "R1" (id 0) (at 134.62 100.965 0)
+    (property "Reference" "R46" (id 0) (at 134.62 100.965 0)
       (effects (font (size 1.27 1.27)) (justify left))
     )
@@
   (symbol (lib_id "Device:R_Small") (at 133.35 107.95 0)
     (in_bom yes) (on_board yes)
-    (property "Reference" "R2" (id 0) (at 134.62 107.95 0)
+    (property "Reference" "R47" (id 0) (at 134.62 107.95 0)
       (effects (font (size 1.27 1.27)) (justify left))
     )
@@
   (symbol (lib_id "Jumper:SolderJumper_3_Open") (at 132.08 86.995 0)
     (in_bom yes) (on_board yes)
-    (property "Reference" "JP3" (id 0) (at 132.08 81.788 0))
+    (property "Reference" "JP7" (id 0) (at 132.08 81.788 0))
     (property "Value" "V_SEL" (id 1) (at 132.08 84.0994 0))
     (property "Footprint" "Jumper:SolderJumper-3_P1.3mm_Open_RoundedPad1.0x1.5mm" (id 2) (at 132.08 86.995 0)
@@
   (symbol (lib_id "Connector_Generic_MountingPin:Conn_01x04_MountingPin") (at 126.365 94.615 0) (mirror y)
     (in_bom yes) (on_board yes)
-    (property "Reference" "J23" (id 0) (at 124.46 94.615 0)
+    (property "Reference" "J15" (id 0) (at 124.46 94.615 0)
       (effects (font (size 1.27 1.27)) (justify left))
     )
@@
   (symbol (lib_id "Device:R_Small") (at 155.575 95.885 90) (mirror x)
     (in_bom yes) (on_board yes)
-    (property "Reference" "R7" (id 0) (at 154.305 93.98 90)
+    (property "Reference" "R48" (id 0) (at 154.305 93.98 90)
       (effects (font (size 1.27 1.27)) (justify right))
     )
@@
   (symbol (lib_id "Device:C_Small") (at 159.385 99.06 0) (mirror y)
     (in_bom yes) (on_board yes)
-    (property "Reference" "C2" (id 0) (at 165.1 98.425 0)
+    (property "Reference" "C53" (id 0) (at 165.1 98.425 0)
       (effects (font (size 1.27 1.27)) (justify left))
     )
