File: PyroOutput.kicad_sch (KiCad schematic)
At the start: 9 parts, among them J11 Pyro, U11 TPS1HC100

Commit message: WIP v1.1, fixed JP2 footprint, replaced STM footprint, re-routing in progress
Parts:
- renumbered C45 to C61, D8 to D12, J11 to J22, R32 to R66, R33 to R67, R34 to R68, R35 to R69, R36 to R70, U11 to U19
Changed lines of the file:
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@@
   (symbol (lib_id "Device:R_Small") (at 160.02 113.03 180)
     (in_bom yes) (on_board yes)
-    (property "Reference" "R35" (id 0) (at 161.29 112.395 0)
+    (property "Reference" "R69" (id 0) (at 161.29 112.395 0)
       (effects (font (size 1.27 1.27)) (justify right))
     )
@@
   (symbol (lib_id "Device:C_Small") (at 127 98.425 270)
     (in_bom yes) (on_board yes)
-    (property "Reference" "C45" (id 0) (at 125.73 95.885 90)
+    (property "Reference" "C61" (id 0) (at 125.73 95.885 90)
       (effects (font (size 1.27 1.27)) (justify left))
     )
@@
   (symbol (lib_id "Device:R_Small") (at 129.54 112.395 0) (mirror x)
     (in_bom yes) (on_board yes)
-    (property "Reference" "R33" (id 0) (at 128.27 111.76 0)
+    (property "Reference" "R67" (id 0) (at 128.27 111.76 0)
       (effects (font (size 1.27 1.27)) (justify right))
     )
@@
   (symbol (lib_id "TXV_LIB:TPS1HC100") (at 144.145 107.315 0)
     (in_bom yes) (on_board yes)
-    (property "Reference" "U11" (id 0) (at 144.145 90.17 0))
+    (property "Reference" "U19" (id 0) (at 144.145 90.17 0))
     (property "Value" "TPS1HC100" (id 1) (at 144.145 92.075 0))
     (property "Footprint" "Package_SO:HTSSOP-14-1EP_4.4x5mm_P0.65mm_EP3.4x5mm_Mask3x3.1mm" (id 2) (at 144.145 123.825 0)
@@
   (symbol (lib_id "Device:R_Small") (at 122.555 106.68 0)
     (in_bom yes) (on_board yes)
-    (property "Reference" "R32" (id 0) (at 119.38 106.045 0))
+    (property "Reference" "R66" (id 0) (at 119.38 106.045 0))
     (property "Value" "120" (id 1) (at 119.38 107.95 0))
     (property "Footprint" "Resistor_SMD:R_0603_1608Metric" (id 2) (at 122.555 106.68 0)
@@
   (symbol (lib_id "Device:R_Small") (at 163.83 92.71 270) (mirror x)
     (in_bom yes) (on_board yes)
-    (property "Reference" "R36" (id 0) (at 161.925 88.9 90)
+    (property "Reference" "R70" (id 0) (at 161.925 88.9 90)
       (effects (font (size 1.27 1.27)) (justify left))
     )
@@
   (symbol (lib_id "Device:R_Small") (at 157.48 92.71 270)
     (in_bom yes) (on_board yes)
-    (property "Reference" "R34" (id 0) (at 157.48 88.9 90))
+    (property "Reference" "R68" (id 0) (at 157.48 88.9 90))
     (property "Value" "56k" (id 1) (at 157.48 90.805 90))
     (property "Footprint" "Resistor_SMD:R_0603_1608Metric" (id 2) (at 157.48 92.71 0)
@@
   (symbol (lib_id "Device:LED_Small_Filled") (at 122.555 112.395 90)
     (in_bom yes) (on_board yes)
-    (property "Reference" "D8" (id 0) (at 116.205 111.76 90)
+    (property "Reference" "D12" (id 0) (at 116.205 111.76 90)
       (effects (font (size 1.27 1.27)) (justify right))
     )
@@
   (symbol (lib_id "Connector_Generic:Conn_01x02") (at 166.37 100.965 0) (mirror x)
     (in_bom yes) (on_board yes)
-    (property "Reference" "J11" (id 0) (at 168.402 100.7618 0)
-      (effects (font (size 1.27 1.27)) (justify left))
-    )
+    (property "Reference" "J22" (id 0) (at 168.402 100.7618 0)
+      (effects (font (size 1.27 1.27)) (justify left))
+    )
