File: uHoubolt_PCB_ECU.kicad_sch (KiCad schematic)
At the start: 86 parts, among them J1 Power In, J2 Debug, J3 CAN1, J35 CAN1, J36 CAN2, J37 CAN1, J38 CAN2, J4 CAN2, J5 CAN1, J6 CAN2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

Commit message: WIP v1.1, fixed JP2 footprint, replaced STM footprint, re-routing in progress
Parts:
- U6: footprint Package_QFP:LQFP-80_14x14mm_P0.65mm -> Package_QFP:LQFP-80_12x12mm_P0.5mm
Changed lines of the file:
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@@
     (property "Reference" "U6" (id 0) (at 75.565 146.685 0))
     (property "Value" "STM32G491MET6-LQFP80" (id 1) (at 75.565 167.64 90))
-    (property "Footprint" "Package_QFP:LQFP-80_14x14mm_P0.65mm" (id 2) (at 76.835 177.8 90)
+    (property "Footprint" "Package_QFP:LQFP-80_12x12mm_P0.5mm" (id 2) (at 76.835 177.8 90)
       (effects (font (size 1.27 1.27)) hide)
     )
@@
     )
     (path "/00000000-0000-0000-0000-000063229df9"
-      (reference "U6") (unit 1) (value "STM32G491MET6-LQFP80") (footprint "Package_QFP:LQFP-80_14x14mm_P0.65mm")
+      (reference "U6") (unit 1) (value "STM32G491MET6-LQFP80") (footprint "Package_QFP:LQFP-80_12x12mm_P0.5mm")
     )
     (path "/00000000-0000-0000-0000-000060ab74cf"
